File: transit.kicad_pcb (KiCad board)
At the start: 2 copper layers, 210 x 300 mm, 376 parts, among them J1 USB_C_Receptacle_USB2.0_16P, J2 Conn_01x03, SW1 RESET, SW2 BOOT, U1 ESP32-C3-MINI-1, U2 SPX3819M5-L-3-3, U3 USBLC6-2SC6, U4 SN74LVC8T245PWR, U5 TPU3013S5, U6 BH1603FVC-TR

Commit message: PCBA prototype order
Parts:
- removed REF** (x39): Untitled, EasyEDA:rail_station
- removed REF** (x13): Untitled, EasyEDA:Ferry port
- C11: renamed from C8; footprint EasyEDA:C0805 -> EasyEDA:C0603
- C12: renamed from C9; footprint EasyEDA:C0805 -> EasyEDA:C0603
- C15: renamed from C12; footprint EasyEDA:C0805 -> EasyEDA:C0603
- C8: renamed from C13; footprint EasyEDA:C0805 -> EasyEDA:C0603
- LED401: renamed from LED14; value Bremerton -> WS2812B-Mini
- LED415: renamed from LED27; value Seattle (Bremerton) -> WS2812B-Mini
- LED416: renamed from LED28; value Westlake Center -> WS2812B-2020
- LED420: renamed from LED32; value Seattle Center -> WS2812B-2020
- LED421: renamed from LED33; value Seattle (Bainbridge) -> WS2812B-Mini
- LED433: renamed from LED42; value Bainbridge -> WS2812B-Mini
- LED434: renamed from LED43; value Kingston -> WS2812B-Mini
- LED447: renamed from LED56; value Edmonds -> WS2812B-Mini
- LED501: renamed from LED400; value Port_Defiance -> WS2812B-Mini
- LED507: renamed from LED404; value Tahlequah -> WS2812B-Mini
- LED508: renamed from LED405; value Vashon_Island -> WS2812B-Mini
- LED513: renamed from LED408; value Southworth -> WS2812B-Mini
- LED525: renamed from LED417; value Fauntleroy -> WS2812B-Mini
- LED544: renamed from LED432; value Seattle (Vashon) -> WS2812B-Mini
- LED547: renamed from LED435; value West Seattle -> WS2812B-Mini
- SW1: value RESET -> SW_SPST
- SW2: value BOOT -> SW_SPST
- moved C601 9.17 mm to (182.4, -57.2), turned to 135 degrees
- moved C401 3.51 mm to (118.4, 51.0), turned to 180 degrees
- moved C402 2.64 mm to (126.0, -33.2), turned to 180 degrees
- moved C201 1.91 mm to (151.4, 200.1)
- moved C501 1.42 mm to (75.4, 187.3)
- moved C1 0.46 mm to (211.7, 158.3)
- moved C2 0.36 mm to (211.2, 160.4)
- moved R1 0.36 mm to (211.2, 162.2)
- renumbered C7 to C10, C10 to C13, C11 to C14, C18 to C401, C19 to C402, C16 to C501, C17 to C502, C15 to C6, C14 to C7, C6 to C9, LED223 to LED222, LED224 to LED223, LED225 to LED224, LED226 to LED225, LED227 to LED226, LED228 to LED227, LED229 to LED228, LED230 to LED229, LED231 to LED230, LED232 to LED231, LED233 to LED232, LED234 to LED233, LED235 to LED234, LED236 to LED235, LED237 to LED236, LED238 to LED237, LED239 to LED238, LED240 to LED239, LED241 to LED240, LED242 to LED241, LED243 to LED242, LED244 to LED243, LED245 to LED244, LED246 to LED245, LED247 to LED246, LED248 to LED247, LED249 to LED248, LED250 to LED249, LED251 to LED250, LED252 to LED251, LED253 to LED252, LED254 to LED253, LED306 to LED301, LED312 to LED302, LED318 to LED303, LED324 to LED304, LED329 to LED305, LED334 to LED306, LED339 to LED307, LED344 to LED308, LED349 to LED309, LED354 to LED310, LED304 to LED311, LED310 to LED312, LED316 to LED313, LED322 to LED314, LED327 to LED315, LED332 to LED316, LED337 to LED317, LED342 to LED318, LED347 to LED319, LED352 to LED320, LED305 to LED321, LED311 to LED322, LED317 to LED323, LED323 to LED324, LED328 to LED325, LED333 to LED326, LED338 to LED327, LED343 to LED328, LED348 to LED329, LED353 to LED330, LED303 to LED331, LED309 to LED332, LED315 to LED333, LED321 to LED334, LED326 to LED335, LED331 to LED336, LED336 to LED337, LED341 to LED338, LED346 to LED339, LED351 to LED340, LED301 to LED341, LED307 to LED342, LED313 to LED343, LED320 to LED344, LED325 to LED345, LED330 to LED346, LED335 to LED347, LED340 to LED348, LED13 to LED402, LED23 to LED403, LED22 to LED404, LED21 to LED405, LED44 to LED406, LED19 to LED407, LED18 to LED408, LED17 to LED409, LED16 to LED410, LED15 to LED411, LED25 to LED412, LED26 to LED413, LED439 to LED414, LED29 to LED417, LED30 to LED418, LED31 to LED419, LED41 to LED422, LED40 to LED423, LED39 to LED424, LED38 to LED425, LED37 to LED426, LED36 to LED427, LED35 to LED428, LED34 to LED429, LED437 to LED431, LED436 to LED432, LED53 to LED435, LED52 to LED436, LED51 to LED437, LED50 to LED438, LED49 to LED439, LED48 to LED440, LED47 to LED441, LED46 to LED442, LED45 to LED443, LED55 to LED444, LED54 to LED445, LED438 to LED446, LED401 to LED502, LED402 to LED503, LED403 to LED504, LED4031 to LED505, LED5 to LED506, LED406 to LED509, LED407 to LED510, LED3 to LED511, LED4 to LED512, LED409 to LED514, LED410 to LED515, LED411 to LED516, LED412 to LED517, LED413 to LED518, LED414 to LED519, LED415 to LED520, LED416 to LED521, LED6 to LED522, LED7 to LED523, LED8 to LED524, LED418 to LED526, LED419 to LED527, LED420 to LED528, LED421 to LED529, LED422 to LED530, LED423 to LED531, LED424 to LED532, LED425 to LED533, LED426 to LED534, LED427 to LED535, LED9 to LED536, LED10 to LED537, LED428 to LED538, LED429 to LED539, LED430 to LED540, LED431 to LED541, LED11 to LED542, LED12 to LED543, LED433 to LED545, LED434 to LED546, LED606 to LED601, LED612 to LED602, LED618 to LED603, LED624 to LED604, LED629 to LED605, LED634 to LED606, LED639 to LED607, LED644 to LED608, LED649 to LED609, LED654 to LED610, LED604 to LED611, LED610 to LED612, LED616 to LED613, LED622 to LED614, LED627 to LED615, LED632 to LED616, LED637 to LED617, LED642 to LED618, LED647 to LED619, LED652 to LED620, LED605 to LED621, LED611 to LED622, LED617 to LED623, LED623 to LED624, LED628 to LED625, LED633 to LED626, LED638 to LED627, LED643 to LED628, LED648 to LED629, LED653 to LED630, LED603 to LED631, LED609 to LED632, LED621 to LED633, LED626 to LED634, LED631 to LED635, LED641 to LED637, LED646 to LED638, LED651 to LED639, LED601 to LED640, LED607 to LED641, LED613 to LED642, LED620 to LED643, LED625 to LED644, LED630 to LED645, LED635 to LED646, LED640 to LED647, LED645 to LED648, LED650 to LED649, LED602 to LED650, LED608 to LED651, LED614 to LED652, LED619 to LED653
Connections:
- net Net-(J1-CC1) renamed /USBCC1
- net Net-(J1-CC2) renamed /USBCC2
- LED246 pad 4: unconnected-(LED247-VDD-Pad4) -> +VLED
- LED247 pad 4: unconnected-(LED248-VDD-Pad4) -> +VLED
- LED248 pad 4: unconnected-(LED249-VDD-Pad4) -> +VLED
- LED249 pad 4: unconnected-(LED250-VDD-Pad4) -> +VLED
Routing:
- net Rail W Southbound: track 2.62 -> 7.83 mm, vias 0 -> 2
- net +VLED: track 802.9 -> 799.1 mm
- net GND: track 375.7 -> 378.6 mm, vias 348 -> 347
Other:
- board text added: "Designed in Seattle, for the opening of the Crosslake Connection on March 28, 2026 Hardware design: Michael Benedict Vector art: Eric Benedict Special thanks: @seattlefoodgeek © 2026 Charles Street Labs"
- board text added: "Lynnwood City Center"
- board text added: "Pinehurst"
- board text removed: "Designed in Seattle, for the opening of the Crosslake Connection on March 28, 2026 Hardware design: Michael Benedict Vector art: Eric Benedict Special thanks: @seattlefoodgeek © Charles Street Labs, 2026"
- board text removed: "Lynwood City Center"
- board text removed: "Pinehurst/NE 130th St"
- board text removed: "Seattle Transit"
