File: ferries_s.kicad_sch (KiCad schematic)
At the start: 49 parts

Commit message: PCBA prototype order
Parts:
- LED501: value Port_Defiance -> WS2812B-Mini; Ferry Port (none) -> Port_Defiance
- LED507: value Tahlequah -> WS2812B-Mini; Ferry Port (none) -> Tahlequah
- LED508: value Vashon_Island -> WS2812B-Mini; Ferry Port (none) -> Vashon_Island
- LED513: value Southworth -> WS2812B-Mini; Ferry Port (none) -> Southworth
- LED525: value Fauntleroy -> WS2812B-Mini; Ferry Port (none) -> Fauntleroy
- LED544: value Seattle (Vashon) -> WS2812B-Mini; Ferry Port (none) -> Seattle (Vashon)
- LED547: value West Seattle -> WS2812B-Mini; Ferry Port (none) -> West Seattle
- renumbered C16 to C501, C501 to C502
Other:
- moved on the sheet: C502
Changed lines of the file:
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@@
 	)
 	(junction
-		(at 149.86 35.56)
-		(diameter 0)
-		(color 0 0 0 0)
-	)
-	(junction
 		(at 58.42 57.15)
 		(diameter 0)
@@
 	)
 	(junction
-		(at 110.49 35.56)
-		(diameter 0)
-		(color 0 0 0 0)
-	)
-	(junction
 		(at 54.61 158.75)
 		(diameter 0)
@@
 	)
 	(junction
-		(at 129.54 35.56)
-		(diameter 0)
-		(color 0 0 0 0)
-	)
-	(junction
 		(at 41.91 77.47)
 		(diameter 0)
@@
 	(wire
 		(pts
-			(xy 40.64 99.06) (xy 43.18 99.06)
+			(xy 40.64 99.06) (xy 45.72 99.06)
 		)
 		(stroke
@@
 	(wire
 		(pts
-			(xy 43.18 91.44) (xy 49.53 91.44)
+			(xy 45.72 91.44) (xy 53.34 91.44)
 		)
 		(stroke
@@
 	(wire
 		(pts
-			(xy 43.18 99.06) (xy 43.18 91.44)
+			(xy 45.72 99.06) (xy 45.72 91.44)
 		)
 		(stroke
@@
 	(wire
 		(pts
-			(xy 110.49 35.56) (xy 113.03 35.56)
-		)
-		(stroke
-			(width 0)
-			(type default)
-		)
-	)
-	(wire
-		(pts
 			(xy 139.7 77.47) (xy 139.7 78.74)
 		)
@@
 	(wire
 		(pts
-			(xy 129.54 35.56) (xy 130.81 35.56)
-		)
-		(stroke
-			(width 0)
-			(type default)
-		)
-	)
-	(wire
-		(pts
 			(xy 217.17 77.47) (xy 217.17 78.74)
 		)
@@
 	(wire
 		(pts
-			(xy 149.86 35.56) (xy 151.13 35.56)
-		)
-		(stroke
-			(width 0)
-			(type default)
-		)
-	)
-	(wire
-		(pts
 			(xy 78.74 160.02) (xy 78.74 161.29)
 		)
@@
 			)
 		)
-		(property "Value" "Seattle (Vashon)"
+		(property "Value" "WS2812B-Mini"
 			(at 43.18 154.686 0)
 			(effects
@@
 					(size 1.27 1.27)
 				)
+				(hide yes)
 			)
 		)
@@
 			)
 		)
+		(property "Ferry Port" "Seattle (Vashon)"
+			(at 43.18 154.94 0)
+			(effects
+				(font
+					(size 1.27 1.27)
+				)
+			)
+		)
 		(pin "1"
 		)
@@
 			)
 		)
-		(property "Value" "Port_Defiance"
+		(property "Value" "WS2812B-Mini"
 			(at 59.69 31.496 0)
 			(effects
@@
 					(size 1.27 1.27)
 				)
+				(hide yes)
 			)
 		)
@@
 			)
 		)
+		(property "Ferry Port" "Port_Defiance"
+			(at 60.96 31.75 0)
+			(effects
+				(font
+					(size 1.27 1.27)
+				)
+			)
+		)
 		(pin "1"
 		)
@@
 		(lib_name "CL21B106KOQNNNE_4")
 		(lib_id "EasyEDA:CL21B106KOQNNNE")
-		(at 46.99 90.17 90)
+		(at 50.8 90.17 90)
 		(mirror x)
 		(unit 1)
@@
 		(on_board yes)
 		(dnp no)
-		(property "Reference" "C501"
-			(at 46.99 97.79 90)
+		(property "Reference" "C502"
+			(at 50.8 97.79 90)
 			(effects
 				(font
@@
 		)
 		(property "Value" "150u"
-			(at 48.895 93.98 90)
+			(at 52.705 93.98 90)
 			(effects
 				(font
@@
 		)
 		(property "Footprint" "EasyEDA:CAP-SMD_L3.5-W2.8"
-			(at 57.15 90.17 0)
+			(at 60.96 90.17 0)
 			(effects
 				(font
@@
 		)
 		(property "Datasheet" "https://www.lcsc.com/datasheet/C212682.pdf"
-			(at 59.69 90.17 0)
+			(at 63.5 90.17 0)
 			(effects
 				(font
@@
 		)
 		(property "Description" "150uF ±20% 6.3V Tantalum Capacitors 35mΩ@100kHz CASE-B-3528-21(mm)"
-			(at 46.99 90.17 0)
+			(at 50.8 90.17 0)
 			(effects
 				(font
@@
 		)
 		(property "LCSC Part" "C212682"
-			(at 62.23 90.17 0)
+			(at 66.04 90.17 0)
 			(effects
 				(font
@@
 			(project "transit"
 				(path "/3763eade-a8c8-4ec0-9cf2-9db4442b4ee5/82c886e4-22b8-4801-83ce-05f3d739a980"
-					(reference "C501")
+					(reference "C502")
 					(unit 1)
 				)
@@
 			)
 		)
-		(property "Value" "Fauntleroy"
+		(property "Value" "WS2812B-Mini"
 			(at 30.48 108.966 0)
 			(effects
@@
 					(size 1.27 1.27)
 				)
+				(hide yes)
 			)
 		)
@@
 			)
 		)
+		(property "Ferry Port" "Fauntleroy"
+			(at 30.48 109.22 0)
+			(effects
+				(font
+					(size 1.27 1.27)
+				)
+			)
+		)
 		(pin "1"
 		)
@@
 			)
 		)
-		(property "Value" "Tahlequah"
+		(property "Value" "WS2812B-Mini"
 			(at 180.34 31.496 0)
 			(effects
@@
 					(size 1.27 1.27)
 				)
+				(hide yes)
 			)
 		)
@@
 			)
 		)
+		(property "Ferry Port" "Tahlequah"
+			(at 180.34 31.75 0)
+			(effects
+				(font
+					(size 1.27 1.27)
+				)
+			)
+		)
 		(pin "1"
 		)
@@
 		(on_board yes)
 		(dnp no)
-		(property "Reference" "C16"
+		(property "Reference" "C501"
 			(at 21.59 30.48 90)
 			(effects
@@
 			(project "transit"
 				(path "/3763eade-a8c8-4ec0-9cf2-9db4442b4ee5/82c886e4-22b8-4801-83ce-05f3d739a980"
-					(reference "C16")
+					(reference "C501")
 					(unit 1)
 				)
@@
 			)
 		)
-		(property "Value" "Vashon_Island"
+		(property "Value" "WS2812B-Mini"
 			(at 46.99 53.086 0)
 			(effects
@@
 			)
 		)
+		(property "Ferry Port" "Vashon_Island"
+			(at 57.15 54.61 0)
+			(effects
+				(font
+					(size 1.27 1.27)
+				)
+				(hide yes)
+			)
+		)
 		(pin "1"
 		)
@@
 	(symbol
 		(lib_id "power:GND")
-		(at 49.53 101.6 0)
+		(at 53.34 101.6 0)
 		(unit 1)
 		(exclude_from_sim no)
@@
 		(dnp no)
 		(property "Reference" "#PWR0136"
-			(at 49.53 107.95 0)
+			(at 53.34 107.95 0)
 			(effects
 				(font
@@
 		)
 		(property "Value" "GND"
-			(at 49.276 105.918 0)
+			(at 53.086 105.918 0)
 			(effects
 				(font
@@
 		)
 		(property "Footprint" ""
-			(at 49.53 101.6 0)
+			(at 53.34 101.6 0)
 			(effects
 				(font
@@
 		)
 		(property "Datasheet" ""
-			(at 49.53 101.6 0)
+			(at 53.34 101.6 0)
 			(effects
 				(font
@@
 		)
 		(property "Description" "Power symbol creates a global label with name \"GND\" , ground"
-			(at 49.53 101.6 0)
+			(at 53.34 101.6 0)
 			(effects
 				(font
@@
 			)
 		)
-		(property "Value" "West Seattle"
+		(property "Value" "WS2812B-Mini"
 			(at 110.49 154.686 0)
 			(effects
@@
 					(size 1.27 1.27)
 				)
+				(hide yes)
 			)
 		)
@@
 			)
 		)
+		(property "Ferry Port" "West Seattle"
+			(at 110.49 154.94 0)
+			(effects
+				(font
+					(size 1.27 1.27)
+				)
+			)
+		)
 		(pin "1"
 		)
@@
 			)
 		)
-		(property "Value" "Southworth"
+		(property "Value" "WS2812B-Mini"
 			(at 30.48 73.406 0)
 			(effects
@@
 					(size 1.27 1.27)
 				)
+				(hide yes)
 			)
 		)
@@
 			)
 		)
+		(property "Ferry Port" "Southworth"
+			(at 30.48 73.66 0)
+			(effects
+				(font
+					(size 1.27 1.27)
+				)
+			)
+		)

Commit message: Sounder and T silk, before scripting
Parts:
- removed C501: 150u, EasyEDA:CAP-SMD_L3.5-W2.8, symbol EasyEDA:CL21B106KOQNNNE
- removed LED501, LED507: WS2812B-Mini, EasyEDA:LED-SMD_4P-L3.5-W3.5-TL_WS2812B, symbol EasyEDA:WS2812B-MINI
- removed LED502, LED503, LED504, LED505, LED506: WS2812B-2020, EasyEDA:LED-SMD_4P-L2.0-W2.0-TL_WS2812B-2020, symbol EasyEDA:WS2812B-2020

Commit message: layout water taxi
Parts:
- removed C502: 150u, EasyEDA:CAP-SMD_L3.5-W2.8, symbol EasyEDA:CL21B106KOQNNNE
- removed LED508, LED513, LED525, LED544, LED547: WS2812B-Mini, EasyEDA:LED-SMD_4P-L3.5-W3.5-TL_WS2812B, symbol EasyEDA:WS2812B-MINI
- removed LED509, LED510, LED511, LED512, LED514, LED515, LED516, LED517, LED518, LED519, LED520, LED521, LED522, LED523, LED524, LED526, LED527, LED528, LED529, LED530, LED531, LED532, LED533, LED534, LED535, LED536, LED537, LED538, LED539, LED540, LED541, LED542, LED543, LED545, LED546: WS2812B-2020, EasyEDA:LED-SMD_4P-L2.0-W2.0-TL_WS2812B-2020, symbol EasyEDA:WS2812B-2020
Connections:
- no-connect marks 1 -> 0
Other:
- note removed: "Bypass Vashon after 423, continue to Seattle"
