File: ferries.kicad_sch (KiCad schematic)
At the start: 0 parts

Commit message: Sounder and T silk, before scripting
Other:
- added sheet port_defiance_tahlequah (port_defiance_tahlequah.kicad_sch)
Changed lines of the file:
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@@
 	(paper "A4")
+	(sheet
+		(at 64.77 38.1)
+		(size 20.32 5.08)
+		(exclude_from_sim no)
+		(in_bom yes)
+		(on_board yes)
+		(dnp no)
+		(fields_autoplaced yes)
+		(stroke
+			(width 0.1524)
+			(type solid)
+		)
+		(fill
+			(color 0 0 0 0)
+		)
+		(property "Sheetname" "port_defiance_tahlequah"
+			(at 64.77 37.3884 0)
+			(show_name no)
+			(do_not_autoplace no)
+			(effects
+				(font
+					(size 1.27 1.27)
+				)
+				(justify left bottom)
+			)
+		)
+		(property "Sheetfile" "port_defiance_tahlequah.kicad_sch"
+			(at 64.77 43.7646 0)
+			(show_name no)
+			(do_not_autoplace no)
+			(effects
+				(font
+					(size 1.27 1.27)
+				)
+				(justify left top)
+			)
+		)
+		(instances
+			(project "transit"
+				(path "/3763eade-a8c8-4ec0-9cf2-9db4442b4ee5/153adc6e-a3b0-4527-a19a-87e28aab4b4d"
+					(page "3")
+				)
+			)
+		)
+	)
 	(sheet
 		(at 25.4 55.88)

Commit message: layout water taxi
Other:
- added sheet fauntleroy_vashon_southworth (fauntleroy_vashon_southworth.kicad_sch)
- added sheet water_taxi (water_taxi.kicad_sch)
Changed lines of the file:
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@@
 	(paper "A4")
+	(sheet
+		(at 64.77 53.34)
+		(size 20.32 5.08)
+		(exclude_from_sim no)
+		(in_bom yes)
+		(on_board yes)
+		(dnp no)
+		(fields_autoplaced yes)
+		(stroke
+			(width 0.1524)
+			(type solid)
+		)
+		(fill
+			(color 0 0 0 0)
+		)
+		(property "Sheetname" "fauntleroy_vashon_southworth"
+			(at 64.77 52.6284 0)
+			(show_name no)
+			(do_not_autoplace no)
+			(effects
+				(font
+					(size 1.27 1.27)
+				)
+				(justify left bottom)
+			)
+		)
+		(property "Sheetfile" "fauntleroy_vashon_southworth.kicad_sch"
+			(at 64.77 59.0046 0)
+			(show_name no)
+			(do_not_autoplace no)
+			(effects
+				(font
+					(size 1.27 1.27)
+				)
+				(justify left top)
+			)
+		)
+		(instances
+			(project "transit"
+				(path "/3763eade-a8c8-4ec0-9cf2-9db4442b4ee5/153adc6e-a3b0-4527-a19a-87e28aab4b4d"
+					(page "4")
+				)
+			)
+		)
+	)
 	(sheet
 		(at 64.77 38.1)
@@
 				)
 			)
+		)
+	)
+	(sheet
+		(at 66.04 67.31)
+		(size 19.05 5.08)
+		(exclude_from_sim no)
+		(in_bom yes)
+		(on_board yes)
+		(dnp no)
+		(fields_autoplaced yes)
+		(stroke
+			(width 0.1524)
+			(type solid)
+		)
+		(fill
+			(color 0 0 0 0)
+		)
+		(property "Sheetname" "water_taxi"
+			(at 66.04 66.5984 0)
+			(show_name no)
+			(do_not_autoplace no)
+			(effects
+				(font
+					(size 1.27 1.27)
+				)
+				(justify left bottom)
+			)
+		)
+		(property "Sheetfile" "water_taxi.kicad_sch"
+			(at 66.04 72.9746 0)
+			(show_name no)
+			(do_not_autoplace no)
+			(effects
+				(font
+					(size 1.27 1.27)
+				)
+				(justify left top)
+			)
+		)
+		(instances
+			(project "transit"
+				(path "/3763eade-a8c8-4ec0-9cf2-9db4442b4ee5/153adc6e-a3b0-4527-a19a-87e28aab4b4d"
+					(page "5")
+				)
+			)

Commit message: sounder layout checkpoint
Other:
- removed sheet Ferries S
- added sheet edmonds_kingston (edmonds_kingston.kicad_sch)
- added sheet mukilteo_clinton (mukilteo_clinton.kicad_sch)
- added sheet seattle_bainbridge (seattle_bainbridge.kicad_sch)
- added sheet seattle_bremerton (seattle_bremerton.kicad_sch)
- added sheet seattle_kingston (seattle_kingston.kicad_sch)
- added sheet seattle_southworth (seattle_southworth.kicad_sch)

Commit message: route T
Other:
- sheet Ferries N renamed monorail
Changed lines of the file:
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@@
 			(color 0 0 0 0)
 		)
-		(property "Sheetname" "Ferries N"
+		(property "Sheetname" "monorail"
 			(at 25.4 37.3884 0)
 			(show_name no)
@@
 			(project "transit"
 				(path "/3763eade-a8c8-4ec0-9cf2-9db4442b4ee5/153adc6e-a3b0-4527-a19a-87e28aab4b4d"
-					(page "#")
+					(page "20")
 				)
 			)
