File: ferries.kicad_sch (KiCad schematic)
At the start: 0 parts

Commit message: Update README, fix typos
Other:
- sheet port_defiance_tahlequah renamed point_defiance_tahlequah
- sheet point_defiance_tahlequah: file port_defiance_tahlequah.kicad_sch -> point_defiance_tahlequah.kicad_sch
Changed lines of the file:
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@@
 			(color 0 0 0 0)
 		)
-		(property "Sheetname" "port_defiance_tahlequah"
+		(property "Sheetname" "point_defiance_tahlequah"
 			(at 64.77 37.3884 0)
 			(show_name no)
@@
 			)
 		)
-		(property "Sheetfile" "port_defiance_tahlequah.kicad_sch"
+		(property "Sheetfile" "point_defiance_tahlequah.kicad_sch"
 			(at 64.77 43.7646 0)
 			(show_name no)
