File: edmonds_kingston.kicad_sch (KiCad schematic)
At the start: 15 parts

Commit message: Replace ferry port LED
Parts:
- LED1015: value WS2812B-Mini -> WS2812B-MINI-X2; footprint EasyEDA:LED-SMD_4P-L3.5-W3.5-TL_WS2812B -> EasyEDA:LED-SMD_4P-L3.5-W3.5-TL_WS2812B-MINI-X2; symbol EasyEDA:WS2812B-MINI -> EasyEDA:WS2812B-MINI-X2; LCSC Part C527089 -> C4154873
Connections:
- net +VLED: now also LED1015.2 (VDD); no longer LED1015.1 (VDD)
- net EDMONDS_MUKILTEO: now also LED1015.3 (DOUT); no longer LED1015.2 (DOUT)
- net GND: now also LED1015.4 (GND); no longer LED1015.3 (VSS)
- net at LED1014.1 (DO): now also LED1015.1 (DIN); no longer LED1015.4 (DIN)
Changed lines of the file:
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@@
 	)
 	(symbol
-		(lib_id "EasyEDA:WS2812B-MINI")
+		(lib_id "EasyEDA:WS2812B-MINI-X2")
 		(at 205.74 69.215 0)
 		(mirror y)
@@
 			)
 		)
-		(property "Value" "WS2812B-Mini"
+		(property "Value" "WS2812B-MINI-X2"
 			(at 195.58 66.675 0)
 			(hide yes)
@@
 			)
 		)
-		(property "Footprint" "EasyEDA:LED-SMD_4P-L3.5-W3.5-TL_WS2812B"
+		(property "Footprint" "EasyEDA:LED-SMD_4P-L3.5-W3.5-TL_WS2812B-MINI-X2"
 			(at 205.74 81.915 0)
 			(hide yes)
@@
 			)
 		)
-		(property "Datasheet" "https://lcsc.com/product-detail/Light-Emitting-Diodes-LED_Worldsemi-WS2812B-Mini_C527089.html"
+		(property "Datasheet" "https://www.lcsc.com/datasheet/C4154873.pdf"
 			(at 205.74 84.455 0)
 			(hide yes)
@@
 			)
 		)
-		(property "Description" ""
+		(property "Description" "Worldsemi WS2812B-MINI-X2 addressable RGB LED, 3.5 x 3.5 x 0.95 mm"
 			(at 205.74 69.215 0)
 			(hide yes)
@@
 			)
 		)
-		(property "LCSC Part" "C527089"
+		(property "LCSC Part" "C4154873"
 			(at 205.74 86.995 0)
 			(hide yes)
@@
 			)
 		)
+		(pin "4"
+		)
+		(pin "2"
+		)
 		(pin "3"
 		)
 		(pin "1"
 		)
-		(pin "2"
-		)
-		(pin "4"
-		)
 		(instances
