File: fauntleroy_vashon_southworth.kicad_sch (KiCad schematic)
At the start: 26 parts

Commit message: Replace ferry port LED
Parts:
- LED401, LED406, LED419: value WS2812B-Mini -> WS2812B-MINI-X2; footprint EasyEDA:LED-SMD_4P-L3.5-W3.5-TL_WS2812B -> EasyEDA:LED-SMD_4P-L3.5-W3.5-TL_WS2812B-MINI-X2; symbol EasyEDA:WS2812B-MINI -> EasyEDA:WS2812B-MINI-X2; LCSC Part C527089 -> C4154873
Connections:
- net +VLED: now also LED401.2 (VDD), LED406.2 (VDD), LED419.2 (VDD); no longer LED401.1 (VDD), LED406.1 (VDD), LED419.1 (VDD)
- net GND: now also LED401.4 (GND), LED406.4 (GND), LED419.4 (GND); no longer LED401.3 (VSS), LED406.3 (VSS), LED419.3 (VSS)
- net TAHLEQUAH_VASHON: now also LED401.1 (DIN); no longer LED401.4 (DIN)
- net at LED420.3 (DI): now also LED419.3 (DOUT); no longer LED419.2 (DOUT)
- net at LED418.1 (DO): now also LED419.1 (DIN); no longer LED419.4 (DIN)
- net at LED405.1 (DO): now also LED406.1 (DIN); no longer LED406.4 (DIN)
- net at LED402.3 (DI): now also LED401.3 (DOUT); no longer LED401.2 (DOUT)
- net at LED407.3 (DI): now also LED406.3 (DOUT); no longer LED406.2 (DOUT)
Changed lines of the file:
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@@
 	)
 	(symbol
-		(lib_id "EasyEDA:WS2812B-MINI")
+		(lib_id "EasyEDA:WS2812B-MINI-X2")
 		(at 275.59 50.8 0)
 		(mirror y)
@@
 			)
 		)
-		(property "Value" "WS2812B-Mini"
+		(property "Value" "WS2812B-MINI-X2"
 			(at 265.43 49.276 0)
 			(hide yes)
@@
 			)
 		)
-		(property "Footprint" "EasyEDA:LED-SMD_4P-L3.5-W3.5-TL_WS2812B"
+		(property "Footprint" "EasyEDA:LED-SMD_4P-L3.5-W3.5-TL_WS2812B-MINI-X2"
 			(at 275.59 63.5 0)
 			(hide yes)
@@
 			)
 		)
-		(property "Datasheet" "https://lcsc.com/product-detail/Light-Emitting-Diodes-LED_Worldsemi-WS2812B-Mini_C527089.html"
+		(property "Datasheet" "https://www.lcsc.com/datasheet/C4154873.pdf"
 			(at 275.59 66.04 0)
 			(hide yes)
@@
 			)
 		)
-		(property "Description" ""
+		(property "Description" "Worldsemi WS2812B-MINI-X2 addressable RGB LED, 3.5 x 3.5 x 0.95 mm"
 			(at 275.59 50.8 0)
 			(hide yes)
@@
 			)
 		)
-		(property "LCSC Part" "C527089"
+		(property "LCSC Part" "C4154873"
 			(at 275.59 68.58 0)
 			(hide yes)
@@
 			)
 		)
-		(pin "1"
-		)
-		(pin "4"
-		)
 		(pin "2"
 		)
+		(pin "1"
+		)
 		(pin "3"
 		)
+		(pin "4"
+		)
 		(instances
 			(project "transit"
@@
 	)
 	(symbol
-		(lib_id "EasyEDA:WS2812B-MINI")
+		(lib_id "EasyEDA:WS2812B-MINI-X2")
 		(at 172.085 26.67 0)
 		(mirror y)
@@
 			)
 		)
-		(property "Value" "WS2812B-Mini"
+		(property "Value" "WS2812B-MINI-X2"
 			(at 161.925 25.146 0)
 			(hide yes)
@@
 			)
 		)
-		(property "Footprint" "EasyEDA:LED-SMD_4P-L3.5-W3.5-TL_WS2812B"
+		(property "Footprint" "EasyEDA:LED-SMD_4P-L3.5-W3.5-TL_WS2812B-MINI-X2"
 			(at 172.085 39.37 0)
 			(hide yes)
@@
 			)
 		)
-		(property "Datasheet" "https://lcsc.com/product-detail/Light-Emitting-Diodes-LED_Worldsemi-WS2812B-Mini_C527089.html"
+		(property "Datasheet" "https://www.lcsc.com/datasheet/C4154873.pdf"
 			(at 172.085 41.91 0)
 			(hide yes)
@@
 			)
 		)
-		(property "Description" ""
+		(property "Description" "Worldsemi WS2812B-MINI-X2 addressable RGB LED, 3.5 x 3.5 x 0.95 mm"
 			(at 172.085 26.67 0)
 			(hide yes)
@@
 			)
 		)
-		(property "LCSC Part" "C527089"
+		(property "LCSC Part" "C4154873"
 			(at 172.085 44.45 0)
 			(hide yes)
@@
 			)
 		)
-		(pin "1"
-		)
-		(pin "4"
-		)
 		(pin "2"
 		)
+		(pin "1"
+		)
 		(pin "3"
 		)
+		(pin "4"
+		)
 		(instances
 			(project "transit"
@@
 	)
 	(symbol
-		(lib_id "EasyEDA:WS2812B-MINI")
+		(lib_id "EasyEDA:WS2812B-MINI-X2")
 		(at 65.405 26.67 0)
 		(mirror y)
@@
 			)
 		)
-		(property "Value" "WS2812B-Mini"
+		(property "Value" "WS2812B-MINI-X2"
 			(at 55.245 25.146 0)
 			(show_name no)
@@
 			)
 		)
-		(property "Footprint" "EasyEDA:LED-SMD_4P-L3.5-W3.5-TL_WS2812B"
+		(property "Footprint" "EasyEDA:LED-SMD_4P-L3.5-W3.5-TL_WS2812B-MINI-X2"
 			(at 65.405 39.37 0)
 			(hide yes)
@@
 			)
 		)
-		(property "Datasheet" "https://lcsc.com/product-detail/Light-Emitting-Diodes-LED_Worldsemi-WS2812B-Mini_C527089.html"
+		(property "Datasheet" "https://www.lcsc.com/datasheet/C4154873.pdf"
 			(at 65.405 41.91 0)
 			(hide yes)
@@
 			)
 		)
-		(property "Description" ""
+		(property "Description" "Worldsemi WS2812B-MINI-X2 addressable RGB LED, 3.5 x 3.5 x 0.95 mm"
 			(at 65.405 26.67 0)
 			(hide yes)
@@
 			)
 		)
-		(property "LCSC Part" "C527089"
+		(property "LCSC Part" "C4154873"
 			(at 65.405 44.45 0)
 			(hide yes)
@@
 			)
 		)
-		(pin "1"
-		)
-		(pin "4"
-		)
 		(pin "2"
 		)
+		(pin "1"
+		)
 		(pin "3"
 		)
+		(pin "4"
+		)
 		(instances
