File: mukilteo_clinton.kicad_sch (KiCad schematic)
At the start: 22 parts

Commit message: checkpoint before label plugin
Parts:
- removed LED1110, LED1111, LED1113, LED1114, LED1115, LED1116, LED1117, LED1118, LED1119, LED1120, LED1121, LED1122: WS2812B-2020, EasyEDA:LED-SMD_4P-L2.0-W2.0-TL_WS2812B-2020, symbol EasyEDA:WS2812B-2020
Connections:
- net at LED1109.1 (DO): now also LED1112.4 (DIN)
Other:
- moved on the sheet: LED1112

Commit message: Add rail labels
Parts:
- renumbered LED1112 to LED1110
Changed lines of the file:
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@@
 		(dnp no)
 		(fields_autoplaced yes)
-		(property "Reference" "LED1112"
+		(property "Reference" "LED1110"
 			(at 109.22 52.07 0)
 			(show_name no)
@@
 			(project "transit"
 				(path "/3763eade-a8c8-4ec0-9cf2-9db4442b4ee5/153adc6e-a3b0-4527-a19a-87e28aab4b4d/9f6e9def-e5c6-4229-90c0-771c2dd67706"
-					(reference "LED1112")
+					(reference "LED1110")
 					(unit 1)
 				)

Commit message: routing complete
Connections:
- net EDMONDS_MUKILTEO: now reaches LED1101.4 (DIN)
- no-connect marks 0 -> 1
Other:
- moved on the sheet: LED1101, LED1102, LED1103, LED1104, LED1105, LED1106, LED1107, LED1108, LED1109, LED1110

Commit message: rev-b validation run
Parts:
- LED1102, LED1103, LED1104, LED1105, LED1106, LED1107, LED1108, LED1109: LCSC Part C965555 -> C52917434
Changed lines of the file:
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@@
 			)
 		)
-		(property "Datasheet" "https://lcsc.com/product-detail/Light-Emitting-Diodes-LED_Worldsemi-WS2812B-2020_C965555.html"
+		(property "Datasheet" "https://lcsc.com/product-detail/Light-Emitting-Diodes-LED_Worldsemi-WS2812B-2020_C52917434.html"
 			(at 128.905 46.355 0)
 			(hide yes)
@@
 			)
 		)
-		(property "LCSC Part" "C965555"
+		(property "LCSC Part" "C52917434"
 			(at 128.905 48.895 0)
 			(hide yes)
@@
 			)
 		)
-		(property "Datasheet" "https://lcsc.com/product-detail/Light-Emitting-Diodes-LED_Worldsemi-WS2812B-2020_C965555.html"
+		(property "Datasheet" "https://lcsc.com/product-detail/Light-Emitting-Diodes-LED_Worldsemi-WS2812B-2020_C52917434.html"
 			(at 90.805 71.755 0)
 			(hide yes)
@@
 			)
 		)
-		(property "LCSC Part" "C965555"
+		(property "LCSC Part" "C52917434"
 			(at 90.805 74.295 0)
 			(hide yes)
@@
 			)
 		)
-		(property "Datasheet" "https://lcsc.com/product-detail/Light-Emitting-Diodes-LED_Worldsemi-WS2812B-2020_C965555.html"
+		(property "Datasheet" "https://lcsc.com/product-detail/Light-Emitting-Diodes-LED_Worldsemi-WS2812B-2020_C52917434.html"
 			(at 153.035 46.355 0)
 			(hide yes)
@@
 			)
 		)
-		(property "LCSC Part" "C965555"
+		(property "LCSC Part" "C52917434"
 			(at 153.035 48.895 0)
 			(hide yes)
@@
 			)
 		)
-		(property "Datasheet" "https://lcsc.com/product-detail/Light-Emitting-Diodes-LED_Worldsemi-WS2812B-2020_C965555.html"
+		(property "Datasheet" "https://lcsc.com/product-detail/Light-Emitting-Diodes-LED_Worldsemi-WS2812B-2020_C52917434.html"
 			(at 85.725 46.355 0)
 			(hide yes)
@@
 			)
 		)
-		(property "LCSC Part" "C965555"
+		(property "LCSC Part" "C52917434"
 			(at 85.725 48.895 0)
 			(hide yes)
@@
 			)
 		)
-		(property "Datasheet" "https://lcsc.com/product-detail/Light-Emitting-Diodes-LED_Worldsemi-WS2812B-2020_C965555.html"
+		(property "Datasheet" "https://lcsc.com/product-detail/Light-Emitting-Diodes-LED_Worldsemi-WS2812B-2020_C52917434.html"
 			(at 219.075 46.355 0)
 			(hide yes)
@@
 			)
 		)
-		(property "LCSC Part" "C965555"
+		(property "LCSC Part" "C52917434"
 			(at 219.075 48.895 0)
 			(hide yes)
@@
 			)
 		)
-		(property "Datasheet" "https://lcsc.com/product-detail/Light-Emitting-Diodes-LED_Worldsemi-WS2812B-2020_C965555.html"
+		(property "Datasheet" "https://lcsc.com/product-detail/Light-Emitting-Diodes-LED_Worldsemi-WS2812B-2020_C52917434.html"
 			(at 197.485 46.355 0)
 			(hide yes)
@@
 			)
 		)
-		(property "LCSC Part" "C965555"
+		(property "LCSC Part" "C52917434"
 			(at 197.485 48.895 0)
 			(hide yes)
@@
 			)
 		)
-		(property "Datasheet" "https://lcsc.com/product-detail/Light-Emitting-Diodes-LED_Worldsemi-WS2812B-2020_C965555.html"
+		(property "Datasheet" "https://lcsc.com/product-detail/Light-Emitting-Diodes-LED_Worldsemi-WS2812B-2020_C52917434.html"
 			(at 107.315 46.355 0)
 			(hide yes)
@@
 			)
 		)
-		(property "LCSC Part" "C965555"
+		(property "LCSC Part" "C52917434"
 			(at 107.315 48.895 0)
 			(hide yes)
@@
 			)
 		)
-		(property "Datasheet" "https://lcsc.com/product-detail/Light-Emitting-Diodes-LED_Worldsemi-WS2812B-2020_C965555.html"
+		(property "Datasheet" "https://lcsc.com/product-detail/Light-Emitting-Diodes-LED_Worldsemi-WS2812B-2020_C52917434.html"
 			(at 174.625 46.355 0)
 			(hide yes)
@@
 			)
 		)
-		(property "LCSC Part" "C965555"
+		(property "LCSC Part" "C52917434"
 			(at 174.625 48.895 0)
 			(hide yes)
