File: mukilteo_clinton.kicad_sch (KiCad schematic)
At the start: 10 parts

Commit message: Replace ferry port LED
Parts:
- LED1101, LED1110: value WS2812B-MINI -> WS2812B-MINI-X2; footprint EasyEDA:LED-SMD_4P-L3.5-W3.5-TL_WS2812B -> EasyEDA:LED-SMD_4P-L3.5-W3.5-TL_WS2812B-MINI-X2; symbol EasyEDA:WS2812B-MINI -> EasyEDA:WS2812B-MINI-X2; LCSC Part C527089 -> C4154873
Connections:
- net +VLED: now also LED1101.2 (VDD), LED1110.2 (VDD); no longer LED1101.1 (VDD), LED1110.1 (VDD)
- net EDMONDS_MUKILTEO: now also LED1101.1 (DIN); no longer LED1101.4 (DIN)
- net GND: now also LED1101.4 (GND), LED1110.4 (GND); no longer LED1101.3 (VSS), LED1110.3 (VSS)
- net at LED1102.3 (DI): now also LED1101.3 (DOUT); no longer LED1101.2 (DOUT)
- net at LED1109.1 (DO): now also LED1110.1 (DIN); no longer LED1110.4 (DIN)
Changed lines of the file:
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@@
 	)
 	(symbol
-		(lib_id "EasyEDA:WS2812B-MINI")
+		(lib_id "EasyEDA:WS2812B-MINI-X2")
 		(at 64.135 31.115 0)
 		(mirror y)
@@
 			)
 		)
-		(property "Value" "WS2812B-MINI"
+		(property "Value" "WS2812B-MINI-X2"
 			(at 53.975 28.575 0)
 			(show_name no)
@@
 			)
 		)
-		(property "Footprint" "EasyEDA:LED-SMD_4P-L3.5-W3.5-TL_WS2812B"
+		(property "Footprint" "EasyEDA:LED-SMD_4P-L3.5-W3.5-TL_WS2812B-MINI-X2"
 			(at 64.135 43.815 0)
 			(hide yes)
@@
 			)
 		)
-		(property "Datasheet" "https://lcsc.com/product-detail/Light-Emitting-Diodes-LED_Worldsemi-WS2812B-Mini_C527089.html"
+		(property "Datasheet" "https://www.lcsc.com/datasheet/C4154873.pdf"
 			(at 64.135 46.355 0)
 			(hide yes)
@@
 			)
 		)
-		(property "Description" ""
+		(property "Description" "Worldsemi WS2812B-MINI-X2 addressable RGB LED, 3.5 x 3.5 x 0.95 mm"
 			(at 64.135 31.115 0)
 			(hide yes)
@@
 			)
 		)
-		(property "LCSC Part" "C527089"
+		(property "LCSC Part" "C4154873"
 			(at 64.135 48.895 0)
 			(hide yes)
@@
 			)
 		)
-		(pin "1"
+		(pin "2"
+		)
+		(pin "1"
+		)
+		(pin "3"
 		)
 		(pin "4"
-		)
-		(pin "2"
-		)
-		(pin "3"
 		)
 		(instances
@@
 	)
 	(symbol
-		(lib_id "EasyEDA:WS2812B-MINI")
+		(lib_id "EasyEDA:WS2812B-MINI-X2")
 		(at 140.335 56.515 0)
 		(mirror y)
@@
 			)
 		)
-		(property "Value" "WS2812B-MINI"
+		(property "Value" "WS2812B-MINI-X2"
 			(at 130.175 53.975 0)
 			(show_name no)
@@
 			)
 		)
-		(property "Footprint" "EasyEDA:LED-SMD_4P-L3.5-W3.5-TL_WS2812B"
+		(property "Footprint" "EasyEDA:LED-SMD_4P-L3.5-W3.5-TL_WS2812B-MINI-X2"
 			(at 140.335 69.215 0)
 			(hide yes)
@@
 			)
 		)
-		(property "Datasheet" "https://lcsc.com/product-detail/Light-Emitting-Diodes-LED_Worldsemi-WS2812B-Mini_C527089.html"
+		(property "Datasheet" "https://www.lcsc.com/datasheet/C4154873.pdf"
 			(at 140.335 71.755 0)
 			(hide yes)
@@
 			)
 		)
-		(property "Description" ""
+		(property "Description" "Worldsemi WS2812B-MINI-X2 addressable RGB LED, 3.5 x 3.5 x 0.95 mm"
 			(at 140.335 56.515 0)
 			(hide yes)
@@
 			)
 		)
-		(property "LCSC Part" "C527089"
+		(property "LCSC Part" "C4154873"
 			(at 140.335 74.295 0)
 			(hide yes)
@@
 			)
 		)
-		(pin "1"
+		(pin "2"
+		)
+		(pin "1"
+		)
+		(pin "3"
 		)
 		(pin "4"
 		)
-		(pin "2"
-		)
-		(pin "3"
-		)
-		(instances
+		(instances
