File: rail.kicad_sch (KiCad schematic)
At the start: 0 parts

Commit message: sounder layout checkpoint
Other:
- added sheet sounder_n (sounder_n.kicad_sch)
- added sheet sounder_s (sounder_s.kicad_sch)
Changed lines of the file:
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@@
+	)
+	(sheet
+		(at 27.94 88.9)
+		(size 24.13 5.08)
+		(exclude_from_sim no)
+		(in_bom yes)
+		(on_board yes)
+		(dnp no)
+		(fields_autoplaced yes)
+		(stroke
+			(width 0.1524)
+			(type solid)
+		)
+		(fill
+			(color 0 0 0 0)
+		)
+		(property "Sheetname" "sounder_s"
+			(at 27.94 88.1884 0)
+			(show_name no)
+			(do_not_autoplace no)
+			(effects
+				(font
+					(size 1.27 1.27)
+				)
+				(justify left bottom)
+			)
+		)
+		(property "Sheetfile" "sounder_s.kicad_sch"
+			(at 27.94 94.5646 0)
+			(show_name no)
+			(do_not_autoplace no)
+			(effects
+				(font
+					(size 1.27 1.27)
+				)
+				(justify left top)
+			)
+		)
+		(instances
+			(project "transit"
+				(path "/3763eade-a8c8-4ec0-9cf2-9db4442b4ee5/77ee1b5c-3800-46a1-aec6-a1e3c1d3f80f"
+					(page "13")
+				)
+			)
+		)
+	)
+	(sheet
+		(at 27.94 104.14)
+		(size 24.13 5.08)
+		(exclude_from_sim no)
+		(in_bom yes)
+		(on_board yes)
+		(dnp no)
+		(fields_autoplaced yes)
+		(stroke
+			(width 0.1524)
+			(type solid)
+		)
+		(fill
+			(color 0 0 0 0)
+		)
+		(property "Sheetname" "sounder_n"
+			(at 27.94 103.4284 0)
+			(show_name no)
+			(do_not_autoplace no)
+			(effects
+				(font
+					(size 1.27 1.27)
+				)
+				(justify left bottom)
+			)
+		)
+		(property "Sheetfile" "sounder_n.kicad_sch"
+			(at 27.94 109.8046 0)
+			(show_name no)
+			(do_not_autoplace no)
+			(effects
+				(font
+					(size 1.27 1.27)
+				)
+				(justify left top)
+			)
+		)
+		(instances
+			(project "transit"
+				(path "/3763eade-a8c8-4ec0-9cf2-9db4442b4ee5/77ee1b5c-3800-46a1-aec6-a1e3c1d3f80f"
+					(page "14")
+				)
+			)
+		)
 	)
 	(sheet

Commit message: initial layout checkpoint
Other:
- added sheet tacoma_t (tacoma_t.kicad_sch)
Changed lines of the file:
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@@
+	)
+	(sheet
+		(at 27.94 104.14)
+		(size 24.13 5.08)
+		(exclude_from_sim no)
+		(in_bom yes)
+		(on_board yes)
+		(dnp no)
+		(fields_autoplaced yes)
+		(stroke
+			(width 0.1524)
+			(type solid)
+		)
+		(fill
+			(color 0 0 0 0)
+		)
+		(property "Sheetname" "sounder_n"
+			(at 27.94 103.4284 0)
+			(show_name no)
+			(do_not_autoplace no)
+			(effects
+				(font
+					(size 1.27 1.27)
+				)
+				(justify left bottom)
+			)
+		)
+		(property "Sheetfile" "sounder_n.kicad_sch"
+			(at 27.94 109.8046 0)
+			(show_name no)
+			(do_not_autoplace no)
+			(effects
+				(font
+					(size 1.27 1.27)
+				)
+				(justify left top)
+			)
+		)
+		(instances
+			(project "transit"
+				(path "/3763eade-a8c8-4ec0-9cf2-9db4442b4ee5/77ee1b5c-3800-46a1-aec6-a1e3c1d3f80f"
+					(page "14")
+				)
+			)
+		)
+	)
+	(sheet
+		(at 27.94 119.38)
+		(size 24.13 5.08)
+		(exclude_from_sim no)
+		(in_bom yes)
+		(on_board yes)
+		(dnp no)
+		(fields_autoplaced yes)
+		(stroke
+			(width 0.1524)
+			(type solid)
+		)
+		(fill
+			(color 0 0 0 0)
+		)
+		(property "Sheetname" "tacoma_t"
+			(at 27.94 118.6684 0)
+			(show_name no)
+			(do_not_autoplace no)
+			(effects
+				(font
+					(size 1.27 1.27)
+				)
+				(justify left bottom)
+			)
+		)
+		(property "Sheetfile" "tacoma_t.kicad_sch"
+			(at 27.94 125.0446 0)
+			(show_name no)
+			(do_not_autoplace no)
+			(effects
+				(font
+					(size 1.27 1.27)
+				)
+				(justify left top)
+			)
+		)
+		(instances
+			(project "transit"
+				(path "/3763eade-a8c8-4ec0-9db4442b4ee5/77ee1b5c-3800-46a1-aec6-a1e3c1d3f80f"
+					(page "15")
+				)
+			)
+		)
 	)
 	(sheet
@@
 				)
 			)
-		)
-	)
-	(sheet
-		(at 27.94 104.14)
-		(size 24.13 5.08)
-		(exclude_from_sim no)
-		(in_bom yes)
-		(on_board yes)
-		(dnp no)
-		(fields_autoplaced yes)
-		(stroke
-			(width 0.1524)
-			(type solid)
-		)
-		(fill
-			(color 0 0 0 0)
-		)
-		(property "Sheetname" "sounder_n"
-			(at 27.94 103.4284 0)
-			(show_name no)
-			(do_not_autoplace no)
-			(effects
-				(font
-					(size 1.27 1.27)
-				)
-				(justify left bottom)
-			)
-		)
-		(property "Sheetfile" "sounder_n.kicad_sch"
-			(at 27.94 109.8046 0)
-			(show_name no)
-			(do_not_autoplace no)
-			(effects
-				(font
-					(size 1.27 1.27)
-				)
-				(justify left top)
-			)
-		)
-		(instances
-			(project "transit"
-				(path "/3763eade-a8c8-4ec0-9cf2-9db4442b4ee5/77ee1b5c-3800-46a1-aec6-a1e3c1d3f80f"
-					(page "14")
-				)
-			)

Commit message: route link 1
Other:
- sheet Rail E renamed link_2
- sheet Rail W renamed link_1_n
- sheet Rail W Southbound renamed link_1_s
Changed lines of the file:
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@@
 			(color 0 0 0 0)
 		)
-		(property "Sheetname" "Rail E"
+		(property "Sheetname" "link_2"
 			(at 25.4 72.9484 0)
 			(show_name no)
@@
 			(color 0 0 0 0)
 		)
-		(property "Sheetname" "Rail W Southbound"
+		(property "Sheetname" "link_1_s"
 			(at 25.4 55.1684 0)
 			(show_name no)
@@
 			(color 0 0 0 0)
 		)
-		(property "Sheetname" "Rail W"
+		(property "Sheetname" "link_1_n"
 			(at 25.4 37.3884 0)
 			(show_name no)

Commit message: rev-b validation run
Parts:
- added C201, C202: 150u, EasyEDA:CAP-SMD_L3.5-W2.8, symbol EasyEDA:CL21B106KOQNNNE
Connections:
- new net +VLED: C201.1, C202.1
- new net GND: C201.2, C202.2
Other:
- note added: "Bulk capacitors"
