File: rail.kicad_sch (KiCad schematic)
At the start: 2 parts

Commit message: Update BOM, remove VLED bulk capacitors, add Rev C to silkscreen
Parts:
- removed C201, C202: 150u, EasyEDA:CAP-SMD_L3.5-W2.8, symbol EasyEDA:CL21B106KOQNNNE
Other:
- note removed: "Bulk capacitors"
