File: seattle_bremerton.kicad_sch (KiCad schematic)
At the start: 19 parts

Commit message: Replace ferry port LED
Parts:
- LED701, LED719: value WS2812B-Mini -> WS2812B-MINI-X2; footprint EasyEDA:LED-SMD_4P-L3.5-W3.5-TL_WS2812B -> EasyEDA:LED-SMD_4P-L3.5-W3.5-TL_WS2812B-MINI-X2; symbol EasyEDA:WS2812B-MINI -> EasyEDA:WS2812B-MINI-X2; LCSC Part C527089 -> C4154873
Connections:
- net +VLED: now also LED701.2 (VDD), LED719.2 (VDD); no longer LED701.1 (VDD), LED719.1 (VDD)
- net BREMERTON_BAINBRIDGE: now also LED719.3 (DOUT); no longer LED719.2 (DOUT)
- net GND: now also LED701.4 (GND), LED719.4 (GND); no longer LED701.3 (VSS), LED719.3 (VSS)
- net at LED718.1 (DO): now also LED719.1 (DIN); no longer LED719.4 (DIN)
- net at LED702.3 (DI): now also LED701.3 (DOUT); no longer LED701.2 (DOUT)
- net at LED703.1 (DO): now also LED701.1 (DIN); no longer LED701.4 (DIN)
Changed lines of the file:
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@@
 	)
 	(symbol
-		(lib_id "EasyEDA:WS2812B-MINI")
+		(lib_id "EasyEDA:WS2812B-MINI-X2")
 		(at 81.915 66.675 0)
 		(mirror y)
@@
 			)
 		)
-		(property "Value" "WS2812B-Mini"
+		(property "Value" "WS2812B-MINI-X2"
 			(at 71.755 64.135 0)
 			(hide yes)
@@
 			)
 		)
-		(property "Footprint" "EasyEDA:LED-SMD_4P-L3.5-W3.5-TL_WS2812B"
+		(property "Footprint" "EasyEDA:LED-SMD_4P-L3.5-W3.5-TL_WS2812B-MINI-X2"
 			(at 81.915 79.375 0)
 			(hide yes)
@@
 			)
 		)
-		(property "Datasheet" "https://lcsc.com/product-detail/Light-Emitting-Diodes-LED_Worldsemi-WS2812B-Mini_C527089.html"
+		(property "Datasheet" "https://www.lcsc.com/datasheet/C4154873.pdf"
 			(at 81.915 81.915 0)
 			(hide yes)
@@
 			)
 		)
-		(property "Description" ""
+		(property "Description" "Worldsemi WS2812B-MINI-X2 addressable RGB LED, 3.5 x 3.5 x 0.95 mm"
 			(at 81.915 66.675 0)
 			(hide yes)
@@
 			)
 		)
-		(property "LCSC Part" "C527089"
+		(property "LCSC Part" "C4154873"
 			(at 81.915 84.455 0)
 			(hide yes)
@@
 			)
 		)
-		(pin "3"
-		)
-		(pin "1"
+		(pin "4"
 		)
 		(pin "2"
 		)
-		(pin "4"
+		(pin "3"
+		)
+		(pin "1"
 		)
 		(instances
@@
 	)
 	(symbol
-		(lib_id "EasyEDA:WS2812B-MINI")
+		(lib_id "EasyEDA:WS2812B-MINI-X2")
 		(at 200.025 99.06 0)
 		(mirror y)
@@
 			)
 		)
-		(property "Value" "WS2812B-Mini"
+		(property "Value" "WS2812B-MINI-X2"
 			(at 189.865 96.52 0)
 			(hide yes)
@@
 			)
 		)
-		(property "Footprint" "EasyEDA:LED-SMD_4P-L3.5-W3.5-TL_WS2812B"
+		(property "Footprint" "EasyEDA:LED-SMD_4P-L3.5-W3.5-TL_WS2812B-MINI-X2"
 			(at 200.025 111.76 0)
 			(hide yes)
@@
 			)
 		)
-		(property "Datasheet" "https://lcsc.com/product-detail/Light-Emitting-Diodes-LED_Worldsemi-WS2812B-Mini_C527089.html"
+		(property "Datasheet" "https://www.lcsc.com/datasheet/C4154873.pdf"
 			(at 200.025 114.3 0)
 			(hide yes)
@@
 			)
 		)
-		(property "Description" ""
+		(property "Description" "Worldsemi WS2812B-MINI-X2 addressable RGB LED, 3.5 x 3.5 x 0.95 mm"
 			(at 200.025 99.06 0)
 			(hide yes)
@@
 			)
 		)
-		(property "LCSC Part" "C527089"
+		(property "LCSC Part" "C4154873"
 			(at 200.025 116.84 0)
 			(hide yes)
@@
 			)
 		)
-		(pin "3"
-		)
-		(pin "1"
+		(pin "4"
 		)
 		(pin "2"
 		)
-		(pin "4"
+		(pin "3"
+		)
+		(pin "1"
 		)
 		(instances
