File: sounder_n.kicad_sch (KiCad schematic)
At the start: 24 parts

Commit message: route monorail
Connections:
- net MONORAIL_SOUNDER_N: now reaches LED1423.3 (DI)
- net MONORAIL_SOUNDER_N: no longer LED1422.1 (DO)
- new net SOUNDER_N_MONORAIL: LED1422.1 (DO)
Other:
- moved on the sheet: LED1423, LED1424
Changed lines of the file:
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@@
 	(wire
 		(pts
-			(xy 138.43 144.78) (xy 138.43 146.05)
+			(xy 194.945 144.78) (xy 194.945 146.05)
 		)
 		(stroke
@@
 	(wire
 		(pts
-			(xy 133.35 143.51) (xy 133.35 144.78)
+			(xy 189.865 143.51) (xy 189.865 144.78)
 		)
 		(stroke
@@
 	(wire
 		(pts
-			(xy 115.57 144.78) (xy 115.57 146.05)
-		)
-		(stroke
-			(width 0)
-			(type default)
-		)
-	)
-	(wire
-		(pts
 			(xy 87.63 143.51) (xy 87.63 144.78)
 		)
@@
 	(wire
 		(pts
-			(xy 110.49 144.78) (xy 115.57 144.78)
-		)
-		(stroke
-			(width 0)
-			(type default)
-		)
-	)
-	(wire
-		(pts
 			(xy 190.5 114.3) (xy 193.04 114.3)
 		)
@@
 	(wire
 		(pts
-			(xy 156.21 143.51) (xy 158.115 143.51)
+			(xy 212.725 143.51) (xy 214.63 143.51)
 		)
 		(stroke
@@
 	(wire
 		(pts
-			(xy 110.49 143.51) (xy 110.49 144.78)
-		)
-		(stroke
-			(width 0)
-			(type default)
-		)
-	)
-	(wire
-		(pts
 			(xy 156.21 28.575) (xy 156.21 29.845)
 		)
@@
 	(wire
 		(pts
-			(xy 133.35 144.78) (xy 138.43 144.78)
+			(xy 189.865 144.78) (xy 194.945 144.78)
 		)
 		(stroke
@@
 	(wire
 		(pts
-			(xy 113.03 143.51) (xy 115.57 143.51)
+			(xy 169.545 143.51) (xy 172.085 143.51)
 		)
 		(stroke
@@
 	(wire
 		(pts
-			(xy 135.89 143.51) (xy 138.43 143.51)
+			(xy 192.405 143.51) (xy 194.945 143.51)
 		)
 		(stroke
@@
 		)
 	)
+	(global_label "MONORAIL_SOUNDER_N"
+		(shape input)
+		(at 172.085 146.05 180)
+		(fields_autoplaced yes)
+		(effects
+			(font
+				(size 1.27 1.27)
+			)
+			(justify right)
+		)
+		(property "Intersheetrefs" "${INTERSHEET_REFS}"
+			(at 147.5097 146.05 0)
+			(hide yes)
+			(show_name no)
+			(do_not_autoplace no)
+			(effects
+				(font
+					(size 1.27 1.27)
+				)
+				(justify right)
+			)
+		)
+	)
 	(global_label "SOUNDER_S_N"
 		(shape input)
@@
 	(global_label "SOUNDER_N_S"
 		(shape input)
-		(at 158.115 143.51 0)
+		(at 214.63 143.51 0)
+		(fields_autoplaced yes)
+		(effects
+			(font
+				(size 1.27 1.27)
+			)
+			(justify left)
+		)
+		(property "Intersheetrefs" "${INTERSHEET_REFS}"
+			(at 230.9804 143.51 0)
+			(hide yes)
+			(show_name no)
+			(do_not_autoplace no)
+			(effects
+				(font
+					(size 1.27 1.27)
+				)
+				(justify left)
+			)
+		)
+	)
+	(global_label "SOUNDER_N_MONORAIL"
+		(shape input)
+		(at 110.49 143.51 0)
 		(fields_autoplaced yes)
 		(effects
@@
 		)
 		(property "Intersheetrefs" "${INTERSHEET_REFS}"
-			(at 174.4654 143.51 0)
+			(at 135.0653 143.51 0)
 			(hide yes)
 			(show_name no)
@@
 	(symbol
 		(lib_id "power:GND")
-		(at 156.21 146.05 0)
+		(at 212.725 146.05 0)
 		(unit 1)
 		(body_style 1)
@@
 		(dnp no)
 		(property "Reference" "#PWR01440"
-			(at 156.21 152.4 0)
+			(at 212.725 152.4 0)
 			(hide yes)
 			(show_name no)
@@
 		)
 		(property "Value" "GND"
-			(at 155.956 150.368 0)
+			(at 212.471 150.368 0)
 			(show_name no)
 			(do_not_autoplace no)
@@
 		)
 		(property "Footprint" ""
-			(at 156.21 146.05 0)
+			(at 212.725 146.05 0)
 			(hide yes)
 			(show_name no)
@@
 		)
 		(property "Datasheet" ""
-			(at 156.21 146.05 0)
+			(at 212.725 146.05 0)
 			(hide yes)
 			(show_name no)
@@
 		)
 		(property "Description" "Power symbol creates a global label with name \"GND\" , ground"
-			(at 156.21 146.05 0)
+			(at 212.725 146.05 0)
 			(hide yes)
 			(show_name no)
@@
 	(symbol
 		(lib_id "power:VBUS")
-		(at 113.03 143.51 0)
+		(at 169.545 143.51 0)
 		(unit 1)
 		(body_style 1)
@@
 		(dnp no)
 		(property "Reference" "#PWR01437"
-			(at 113.03 147.32 0)
+			(at 169.545 147.32 0)
 			(hide yes)
 			(show_name no)
@@
 		)
 		(property "Value" "+VLED"
-			(at 113.03 139.7 0)
+			(at 169.545 139.7 0)
 			(show_name no)
 			(do_not_autoplace no)
@@
 		)
 		(property "Footprint" ""
-			(at 113.03 143.51 0)
+			(at 169.545 143.51 0)
 			(hide yes)
 			(show_name no)
@@
 		)
 		(property "Datasheet" ""
-			(at 113.03 143.51 0)
+			(at 169.545 143.51 0)
 			(hide yes)
 			(show_name no)
@@
 		)
 		(property "Description" "Power symbol creates a global label with name \"VBUS\""
-			(at 113.03 143.51 0)
+			(at 169.545 143.51 0)
 			(hide yes)
 			(show_name no)
@@
 	(symbol
 		(lib_id "EasyEDA:WS2812B-2020")
-		(at 156.21 140.97 0)
+		(at 212.725 140.97 0)
 		(mirror y)
 		(unit 1)
@@
 		(dnp no)
 		(property "Reference" "LED1424"
-			(at 147.32 135.89 0)
+			(at 203.835 135.89 0)
 			(show_name no)
 			(do_not_autoplace no)
@@
 		)
 		(property "Value" "WS2812B-2020"
-			(at 147.32 138.43 0)
+			(at 203.835 138.43 0)
 			(show_name no)
 			(do_not_autoplace no)
@@
 		)
 		(property "Footprint" "EasyEDA:LED-SMD_4P-L2.0-W2.0-TL_WS2812B-2020"
-			(at 156.21 153.67 0)
+			(at 212.725 153.67 0)
 			(hide yes)
 			(show_name no)
@@
 		)
 		(property "Datasheet" "https://lcsc.com/product-detail/Light-Emitting-Diodes-LED_Worldsemi-WS2812B-2020_C965555.html"
-			(at 156.21 156.21 0)
+			(at 212.725 156.21 0)
 			(hide yes)
 			(show_name no)
@@
 		)
 		(property "Description" ""
-			(at 156.21 140.97 0)
+			(at 212.725 140.97 0)
 			(hide yes)
 			(show_name no)
@@
 		)
 		(property "LCSC Part" "C965555"
-			(at 156.21 158.75 0)
+			(at 212.725 158.75 0)
 			(hide yes)
 			(show_name no)
@@
 	(symbol
 		(lib_id "power:GND")
-		(at 133.35 146.05 0)
+		(at 189.865 146.05 0)
 		(unit 1)
 		(body_style 1)
@@
 		(dnp no)
 		(property "Reference" "#PWR01438"
-			(at 133.35 152.4 0)
+			(at 189.865 152.4 0)
 			(hide yes)
 			(show_name no)
@@
 		)
 		(property "Value" "GND"
-			(at 133.096 150.368 0)
+			(at 189.611 150.368 0)
 			(show_name no)
 			(do_not_autoplace no)
@@
 		)
 		(property "Footprint" ""
-			(at 133.35 146.05 0)
+			(at 189.865 146.05 0)
 			(hide yes)
 			(show_name no)
@@
 		)
 		(property "Datasheet" ""
-			(at 133.35 146.05 0)
+			(at 189.865 146.05 0)
 			(hide yes)
 			(show_name no)
@@
 		)
 		(property "Description" "Power symbol creates a global label with name \"GND\" , ground"
-			(at 133.35 146.05 0)
+			(at 189.865 146.05 0)
 			(hide yes)
 			(show_name no)
@@
 	(symbol
 		(lib_id "EasyEDA:WS2812B-2020")
-		(at 133.35 140.97 0)
+		(at 189.865 140.97 0)
 		(mirror y)
 		(unit 1)
@@
 		(dnp no)
 		(property "Reference" "LED1423"
-			(at 124.46 135.89 0)
+			(at 180.975 135.89 0)
 			(show_name no)
 			(do_not_autoplace no)
@@
 		)
 		(property "Value" "WS2812B-2020"
-			(at 124.46 138.43 0)
+			(at 180.975 138.43 0)
 			(show_name no)
 			(do_not_autoplace no)
@@
 		)
 		(property "Footprint" "EasyEDA:LED-SMD_4P-L2.0-W2.0-TL_WS2812B-2020"
-			(at 133.35 153.67 0)
+			(at 189.865 153.67 0)
 			(hide yes)
 			(show_name no)
@@
 		)
 		(property "Datasheet" "https://lcsc.com/product-detail/Light-Emitting-Diodes-LED_Worldsemi-WS2812B-2020_C965555.html"
-			(at 133.35 156.21 0)
+			(at 189.865 156.21 0)
 			(hide yes)
 			(show_name no)
@@
 		)
 		(property "Description" ""
-			(at 133.35 140.97 0)
+			(at 189.865 140.97 0)
 			(hide yes)
 			(show_name no)
@@
 		)
 		(property "LCSC Part" "C965555"
-			(at 133.35 158.75 0)
+			(at 189.865 158.75 0)
 			(hide yes)
 			(show_name no)
@@
 	(symbol
 		(lib_id "power:VBUS")
-		(at 135.89 143.51 0)
+		(at 192.405 143.51 0)
 		(unit 1)
 		(body_style 1)
@@
 		(dnp no)
 		(property "Reference" "#PWR01439"
-			(at 135.89 147.32 0)
+			(at 192.405 147.32 0)
 			(hide yes)
 			(show_name no)
@@
 		)
 		(property "Value" "+VLED"
-			(at 135.89 139.7 0)
+			(at 192.405 139.7 0)
 			(show_name no)
 			(do_not_autoplace no)
@@
 		)
 		(property "Footprint" ""
-			(at 135.89 143.51 0)
+			(at 192.405 143.51 0)
 			(hide yes)
 			(show_name no)
@@
 		)
 		(property "Datasheet" ""
-			(at 135.89 143.51 0)
+			(at 192.405 143.51 0)
 			(hide yes)
 			(show_name no)
@@
 		)
 		(property "Description" "Power symbol creates a global label with name \"VBUS\""
-			(at 135.89 143.51 0)
+			(at 192.405 143.51 0)
 			(hide yes)
 			(show_name no)

Commit message: rev-b validation run
Parts:
- LED1401, LED1402, LED1403, LED1404, LED1405, LED1406, LED1407, LED1408, LED1409, LED1410, LED1411, LED1412, LED1413, LED1414, LED1415, LED1416, LED1417, LED1418, LED1419, LED1420, LED1421, LED1422, LED1423, LED1424: LCSC Part C965555 -> C52917434
