File: sounder_s.kicad_sch (KiCad schematic)
At the start: 48 parts

Commit message: initial layout checkpoint
Parts:
- renumbered LED1328 to LED1326, LED1331 to LED1327, LED1334 to LED1328, LED1337 to LED1329, LED1339 to LED1330, LED1341 to LED1331, LED1343 to LED1332, LED1345 to LED1333, LED1347 to LED1334, LED1327 to LED1335, LED1330 to LED1336, LED1333 to LED1337, LED1336 to LED1338, LED1338 to LED1339, LED1342 to LED1341, LED1344 to LED1342, LED1346 to LED1343, LED1348 to LED1344, LED1326 to LED1345, LED1329 to LED1346, LED1332 to LED1347, LED1335 to LED1348

Commit message: checkpoint before label plugin
Parts:
- removed LED1301, LED1302, LED1312, LED1317, LED1320, LED1325, LED1326, LED1336, LED1341, LED1344: WS2812B-2020, EasyEDA:LED-SMD_4P-L2.0-W2.0-TL_WS2812B-2020, symbol EasyEDA:WS2812B-2020
Connections:
- net at LED1313.3 (DI): now also LED1311.1 (DO)
- net at LED1343.1 (DO): now also LED1345.3 (DI)
- net at LED1337.3 (DI): now also LED1335.1 (DO)
- net at LED1316.1 (DO): now also LED1318.3 (DI)
- net at LED1342.3 (DI): now also LED1340.1 (DO)
- net at LED1321.3 (DI): now also LED1319.1 (DO)

Commit message: Add rail labels
Parts:
- renumbered LED1303 to LED1301, LED1304 to LED1302, LED1305 to LED1303, LED1306 to LED1304, LED1307 to LED1305, LED1308 to LED1306, LED1309 to LED1307, LED1310 to LED1308, LED1311 to LED1309, LED1313 to LED1310, LED1314 to LED1311, LED1315 to LED1312, LED1316 to LED1313, LED1318 to LED1314, LED1319 to LED1315, LED1321 to LED1316, LED1322 to LED1317, LED1323 to LED1318, LED1324 to LED1319, LED1327 to LED1320, LED1328 to LED1321, LED1329 to LED1322, LED1330 to LED1323, LED1331 to LED1324, LED1332 to LED1325, LED1333 to LED1326, LED1334 to LED1327, LED1335 to LED1328, LED1337 to LED1329, LED1338 to LED1330, LED1339 to LED1331, LED1340 to LED1332, LED1342 to LED1333, LED1343 to LED1334, LED1345 to LED1335, LED1346 to LED1336, LED1347 to LED1337, LED1348 to LED1338

Commit message: route T
Connections:
- net T_SOUNDER: now reaches LED1301.3 (DI)
Changed lines of the file:
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@@
+		)
+	)
+	(global_label "T_SOUNDER"
+		(shape input)
+		(at 76.2 30.48 180)
+		(fields_autoplaced yes)
+		(effects
+			(font
+				(size 1.27 1.27)
+			)
+			(justify right)
+		)
+		(property "Intersheetrefs" "${INTERSHEET_REFS}"
+			(at 62.3896 30.48 0)
+			(hide yes)
+			(show_name no)
+			(do_not_autoplace no)
+			(effects
+				(font
+					(size 1.27 1.27)
+				)
+				(justify right)
+			)
 		)
 	)

Commit message: Renumber Sounder, ready to route
Connections:
- net SOUNDER_S_N: now reaches LED1319.1 (DO)
- net SOUNDER_N_S: now reaches LED1320.3 (DI)
Changed lines of the file:
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@@
-	(wire
-		(pts
-			(xy 77.47 115.57) (xy 82.55 115.57)
-		)
-		(stroke
-			(width 0)
-			(type default)
-		)
-	)
 	(wire
 		(pts
@@
 	(wire
 		(pts
+			(xy 75.565 115.57) (xy 82.55 115.57)
+		)
+		(stroke
+			(width 0)
+			(type default)
+		)
+	)
+	(wire
+		(pts
 			(xy 215.9 29.21) (xy 218.44 29.21)
 		)
@@
 		)
 	)
+	(global_label "SOUNDER_S_N"
+		(shape input)
+		(at 127 80.01 0)
+		(fields_autoplaced yes)
+		(effects
+			(font
+				(size 1.27 1.27)
+			)
+			(justify left)
+		)
+		(property "Intersheetrefs" "${INTERSHEET_REFS}"
+			(at 143.3504 80.01 0)
+			(hide yes)
+			(show_name no)
+			(do_not_autoplace no)
+			(effects
+				(font
+					(size 1.27 1.27)
+				)
+				(justify left)
+			)
+		)
+	)
+	(global_label "SOUNDER_N_S"
+		(shape input)
+		(at 75.565 115.57 180)
+		(fields_autoplaced yes)
+		(effects
+			(font
+				(size 1.27 1.27)
+			)
+			(justify right)
+		)
+		(property "Intersheetrefs" "${INTERSHEET_REFS}"
+			(at 59.2146 115.57 0)
+			(hide yes)
+			(show_name no)
+			(do_not_autoplace no)
+			(effects
+				(font
+					(size 1.27 1.27)
+				)
+				(justify right)
+			)
+		)
+	)

Commit message: route link 1
Connections:
- net LINK_1_N: now reaches LED1338.1 (DO)
Changed lines of the file:
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@@
+		)
+	)
+	(global_label "LINK_1_N"
+		(shape input)
+		(at 128.27 165.1 0)
+		(fields_autoplaced yes)
+		(effects
+			(font
+				(size 1.27 1.27)
+			)
+			(justify left)
+		)
+		(property "Intersheetrefs" "${INTERSHEET_REFS}"
+			(at 139.9638 165.1 0)
+			(hide yes)
+			(show_name no)
+			(do_not_autoplace no)
+			(effects
+				(font
+					(size 1.27 1.27)
+				)
+				(justify left)
+			)
 		)
 	)

Commit message: rev-b validation run
Parts:
- LED1301, LED1302, LED1303, LED1304, LED1305, LED1306, LED1307, LED1308, LED1309, LED1310, LED1311, LED1312, LED1313, LED1314, LED1315, LED1316, LED1317, LED1318, LED1319, LED1320, LED1321, LED1322, LED1323, LED1324, LED1325, LED1326, LED1327, LED1328, LED1329, LED1330, LED1331, LED1332, LED1333, LED1334, LED1335, LED1336, LED1337, LED1338: LCSC Part C965555 -> C52917434
