File: tacoma_t.kicad_sch (KiCad schematic)
At the start: 24 parts

Commit message: route T
Parts:
- renumbered LED1501 to LED1801, LED1502 to LED1802, LED1503 to LED1803, LED1504 to LED1804, LED1505 to LED1805, LED1506 to LED1806, LED1507 to LED1807, LED1508 to LED1808, LED1509 to LED1809, LED1510 to LED1810, LED1511 to LED1811, LED1512 to LED1812, LED1513 to LED1813, LED1514 to LED1814, LED1515 to LED1815, LED1516 to LED1816, LED1517 to LED1817, LED1518 to LED1818, LED1519 to LED1819, LED1520 to LED1820, LED1521 to LED1821, LED1522 to LED1822, LED1523 to LED1823, LED1524 to LED1824
Connections:
- net at LED1812.1 (DO): now also LED1813.3 (DI)
- net Rail W: now reaches LED1801.3 (DI)
- net T_SOUNDER: now reaches LED1824.1 (DO)

Commit message: route link 1
Connections:
- net Rail W renamed RAIL
Changed lines of the file:
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@@
 		)
 	)
-	(global_label "Rail W"
+	(global_label "RAIL"
 		(shape input)
 		(at 33.655 31.75 180)
@@
 		)
 		(property "Intersheetrefs" "${INTERSHEET_REFS}"
-			(at 24.5618 31.75 0)
+			(at 26.6783 31.75 0)
 			(hide yes)
 			(show_name no)

Commit message: rev-b validation run
Parts:
- LED1801, LED1802, LED1803, LED1804, LED1805, LED1806, LED1807, LED1808, LED1809, LED1810, LED1811, LED1812, LED1813, LED1814, LED1815, LED1816, LED1817, LED1818, LED1819, LED1820, LED1821, LED1822, LED1823, LED1824: LCSC Part C965555 -> C52917434
