File: seattle_bainbridge.kicad_sch (KiCad schematic)
At the start: 12 parts

Commit message: Replace ferry port LED
Parts:
- LED801: value WS2812B-Mini -> WS2812B-MINI-X2; footprint EasyEDA:LED-SMD_4P-L3.5-W3.5-TL_WS2812B -> EasyEDA:LED-SMD_4P-L3.5-W3.5-TL_WS2812B-MINI-X2; symbol EasyEDA:WS2812B-MINI -> EasyEDA:WS2812B-MINI-X2; LCSC Part C527089 -> C4154873
Connections:
- net +VLED: now also LED801.2 (VDD); no longer LED801.1 (VDD)
- net BREMERTON_BAINBRIDGE: now also LED801.1 (DIN); no longer LED801.4 (DIN)
- net GND: now also LED801.4 (GND); no longer LED801.3 (VSS)
- net at LED802.3 (DI): now also LED801.3 (DOUT); no longer LED801.2 (DOUT)
Changed lines of the file:
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@@
 	)
 	(symbol
-		(lib_id "EasyEDA:WS2812B-MINI")
+		(lib_id "EasyEDA:WS2812B-MINI-X2")
 		(at 78.74 33.655 0)
 		(mirror y)
@@
 			)
 		)
-		(property "Value" "WS2812B-Mini"
+		(property "Value" "WS2812B-MINI-X2"
 			(at 68.58 31.115 0)
 			(show_name no)
@@
 			)
 		)
-		(property "Footprint" "EasyEDA:LED-SMD_4P-L3.5-W3.5-TL_WS2812B"
+		(property "Footprint" "EasyEDA:LED-SMD_4P-L3.5-W3.5-TL_WS2812B-MINI-X2"
 			(at 78.74 46.355 0)
 			(hide yes)
@@
 			)
 		)
-		(property "Datasheet" "https://lcsc.com/product-detail/Light-Emitting-Diodes-LED_Worldsemi-WS2812B-Mini_C527089.html"
+		(property "Datasheet" "https://www.lcsc.com/datasheet/C4154873.pdf"
 			(at 78.74 48.895 0)
 			(hide yes)
@@
 			)
 		)
-		(property "Description" ""
+		(property "Description" "Worldsemi WS2812B-MINI-X2 addressable RGB LED, 3.5 x 3.5 x 0.95 mm"
 			(at 78.74 33.655 0)
 			(hide yes)
@@
 			)
 		)
-		(property "LCSC Part" "C527089"
+		(property "LCSC Part" "C4154873"
 			(at 78.74 51.435 0)
 			(hide yes)
@@
 			)
 		)
+		(pin "4"
+		)
+		(pin "2"
+		)
 		(pin "3"
 		)
 		(pin "1"
 		)
-		(pin "2"
-		)
-		(pin "4"
-		)
 		(instances
