File: water_taxi.kicad_sch (KiCad schematic)
At the start: 18 parts

Commit message: Replace ferry port LED
Parts:
- LED514, LED518: value WS2812B-Mini -> WS2812B-MINI-X2; footprint EasyEDA:LED-SMD_4P-L3.5-W3.5-TL_WS2812B -> EasyEDA:LED-SMD_4P-L3.5-W3.5-TL_WS2812B-MINI-X2; symbol EasyEDA:WS2812B-MINI -> EasyEDA:WS2812B-MINI-X2; LCSC Part C527089 -> C4154873
Connections:
- net +VLED: now also LED514.2 (VDD), LED518.2 (VDD); no longer LED514.1 (VDD), LED518.1 (VDD)
- net GND: now also LED514.4 (GND), LED518.4 (GND); no longer LED514.3 (VSS), LED518.3 (VSS)
- net WATER_TAXI_SOUTHWORTH: now also LED518.3 (DOUT); no longer LED518.2 (DOUT)
- net at LED515.3 (DI): now also LED514.3 (DOUT); no longer LED514.2 (DOUT)
- net at LED517.1 (DO): now also LED518.1 (DIN); no longer LED518.4 (DIN)
- net at LED513.1 (DO): now also LED514.1 (DIN); no longer LED514.4 (DIN)
Changed lines of the file:
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@@
 	)
 	(symbol
-		(lib_id "EasyEDA:WS2812B-MINI")
+		(lib_id "EasyEDA:WS2812B-MINI-X2")
 		(at 53.34 104.14 0)
 		(mirror y)
@@
 			)
 		)
-		(property "Value" "WS2812B-Mini"
+		(property "Value" "WS2812B-MINI-X2"
 			(at 43.18 102.616 0)
 			(hide yes)
@@
 			)
 		)
-		(property "Footprint" "EasyEDA:LED-SMD_4P-L3.5-W3.5-TL_WS2812B"
+		(property "Footprint" "EasyEDA:LED-SMD_4P-L3.5-W3.5-TL_WS2812B-MINI-X2"
 			(at 53.34 116.84 0)
 			(hide yes)
@@
 			)
 		)
-		(property "Datasheet" "https://lcsc.com/product-detail/Light-Emitting-Diodes-LED_Worldsemi-WS2812B-Mini_C527089.html"
+		(property "Datasheet" "https://www.lcsc.com/datasheet/C4154873.pdf"
 			(at 53.34 119.38 0)
 			(hide yes)
@@
 			)
 		)
-		(property "Description" ""
+		(property "Description" "Worldsemi WS2812B-MINI-X2 addressable RGB LED, 3.5 x 3.5 x 0.95 mm"
 			(at 53.34 104.14 0)
 			(hide yes)
@@
 			)
 		)
-		(property "LCSC Part" "C527089"
+		(property "LCSC Part" "C4154873"
 			(at 53.34 121.92 0)
 			(hide yes)
@@
 			)
 		)
+		(pin "2"
+		)
 		(pin "1"
 		)
+		(pin "3"
+		)
 		(pin "4"
-		)
-		(pin "2"
-		)
-		(pin "3"
 		)
 		(instances
@@
 	)
 	(symbol
-		(lib_id "EasyEDA:WS2812B-MINI")
+		(lib_id "EasyEDA:WS2812B-MINI-X2")
 		(at 152.4 104.14 0)
 		(mirror y)
@@
 			)
 		)
-		(property "Value" "WS2812B-Mini"
+		(property "Value" "WS2812B-MINI-X2"
 			(at 142.24 102.616 0)
 			(hide yes)
@@
 			)
 		)
-		(property "Footprint" "EasyEDA:LED-SMD_4P-L3.5-W3.5-TL_WS2812B"
+		(property "Footprint" "EasyEDA:LED-SMD_4P-L3.5-W3.5-TL_WS2812B-MINI-X2"
 			(at 152.4 116.84 0)
 			(hide yes)
@@
 			)
 		)
-		(property "Datasheet" "https://lcsc.com/product-detail/Light-Emitting-Diodes-LED_Worldsemi-WS2812B-Mini_C527089.html"
+		(property "Datasheet" "https://www.lcsc.com/datasheet/C4154873.pdf"
 			(at 152.4 119.38 0)
 			(hide yes)
@@
 			)
 		)
-		(property "Description" ""
+		(property "Description" "Worldsemi WS2812B-MINI-X2 addressable RGB LED, 3.5 x 3.5 x 0.95 mm"
 			(at 152.4 104.14 0)
 			(hide yes)
@@
 			)
 		)
-		(property "LCSC Part" "C527089"
+		(property "LCSC Part" "C4154873"
 			(at 152.4 121.92 0)
 			(hide yes)
@@
 			)
 		)
+		(pin "2"
+		)
 		(pin "1"
 		)
+		(pin "3"
+		)
 		(pin "4"
 		)
-		(pin "2"
-		)
-		(pin "3"
-		)
 		(instances
