File: point_defiance_tahlequah.kicad_sch (KiCad schematic)
At the start: 7 parts

Commit message: Update README, fix typos
Parts:
- LED301: Ferry Port Port_Defiance -> Point_Defiance
Changed lines of the file:
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@@
 			)
 		)
-		(property "Ferry Port" "Port_Defiance"
+		(property "Ferry Port" "Point_Defiance"
 			(at 77.47 40.64 0)
 			(show_name no)
