File: transit.kicad_sch (KiCad schematic)
At the start: 70 parts, among them J1 USB_C_Receptacle_USB2.0_16P, J2 USB_C_Receptacle_USB2.0_16P, J3 Conn_01x03, SW1 SW_SPST, SW2 SW_SPST, SW3 SW_SPST, U1 ESP32-C3-MINI-1, U2 TLV75733PDYDR, U3 USBLC6-2SC6, U4 TPU3013S5, U5 BH1603FVC-TR, U6 SN74LVC2T45DCUR

Commit message: Update R values to dim indicator LEDs
Parts:
- R12, R18: value 2K2 -> 10K; LCSC C4190 -> (none); LCSC Part (none) -> C25804
- R4: value 2K2 -> 47K; LCSC C4190 -> (none); LCSC Part (none) -> C25819
Changed lines of the file:
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@@
 			)
 		)
-		(property "Value" "2K2"
+		(property "Value" "47K"
 			(at 273.558 28.956 90)
 			(show_name no)
@@
 			)
 		)
-		(property "Datasheet" "https://www.lcsc.com/datasheet/C4190.pdf"
+		(property "Datasheet" "https://www.lcsc.com/product-detail/Chip-Resistor-Surface-Mount_UNI-ROYAL-Uniroyal-Elec-0603WAF4702T5E_C25819.html"
 			(at 271.78 26.67 0)
 			(hide yes)
@@
 			)
 		)
-		(property "Description" "2.2kΩ ±1% 100mW 0603 Thick Film Resistor"
+		(property "Description" "47kΩ ±1% 100mW 0603 Thick Film Resistor"
 			(at 271.78 26.67 0)
 			(hide yes)
@@
 			)
 		)
-		(property "LCSC" "C4190"
+		(property "LCSC Part" "C25819"
 			(at 271.78 26.67 90)
 			(hide yes)
@@
 			)
 		)
-		(property "Value" "2K2"
+		(property "Value" "10K"
 			(at 264.668 150.876 90)
 			(show_name no)
@@
 			)
 		)
-		(property "Datasheet" "https://www.lcsc.com/datasheet/C4190.pdf"
+		(property "Datasheet" "https://lcsc.com/product-detail/Chip-Resistor-Surface-Mount-UniOhm_10KR-1002-1_C25804.html"
 			(at 262.89 148.59 0)
 			(hide yes)
@@
 			)
 		)
-		(property "Description" "2.2kΩ ±1% 100mW 0603 Thick Film Resistor"
+		(property "Description" "10kΩ ±1% 100mW 0603 Thick Film Resistor"
 			(at 262.89 148.59 0)
 			(hide yes)
@@
 			)
 		)
-		(property "LCSC" "C4190"
+		(property "LCSC Part" "C25804"
 			(at 262.89 148.59 90)
 			(hide yes)
@@
 			)
 		)
-		(property "Value" "2K2"
+		(property "Value" "10K"
 			(at 264.668 125.476 90)
 			(show_name no)
@@
 			)
 		)
-		(property "Datasheet" "https://www.lcsc.com/datasheet/C4190.pdf"
+		(property "Datasheet" "https://lcsc.com/product-detail/Chip-Resistor-Surface-Mount-UniOhm_10KR-1002-1_C25804.html"
 			(at 262.89 123.19 0)
 			(hide yes)
@@
 			)
 		)
-		(property "Description" "2.2kΩ ±1% 100mW 0603 Thick Film Resistor"
+		(property "Description" "10kΩ ±1% 100mW 0603 Thick Film Resistor"
 			(at 262.89 123.19 0)
 			(hide yes)
@@
 			)
 		)
-		(property "LCSC" "C4190"
+		(property "LCSC Part" "C25804"
 			(at 262.89 123.19 90)
 			(hide yes)

Commit message: Remove test points, slight shift bremerton LEDs, cleanup around ALS
Parts:
- removed TP12, TP5, TP7, TP8: Ambient-Light-SNS, TestPoint:TestPoint_Keystone_5000-5004_Miniature, symbol Connector:TestPoint
- renumbered TP6 to TP5, TP9 to TP6, TP10 to TP7, TP11 to TP8
Connections:
- net Data_LED: now also R12.2, U1.13 (GPIO1/ADC1_CH1/XTAL_32K_N); no longer R18.2, U1.12 (GPIO0/ADC1_CH0/XTAL_32K_P)
- net WiFi_LED: now also R18.2, U1.12 (GPIO0/ADC1_CH0/XTAL_32K_P); no longer R12.2, U1.13 (GPIO1/ADC1_CH1/XTAL_32K_N)

Commit message: fix indicator led orientation
Parts:
- LED1, LED2, LED3: symbol Device:LED_Small -> Transit:Kento_LED0805_C229x
Connections:
- net GND: now also LED1.2 (K), LED2.2 (K), LED3.2 (K); no longer LED1.1 (K), LED2.1 (K), LED3.1 (K)
- net at R4.1: now also LED1.1 (A); no longer LED1.2 (A)
- net at R18.1: now also LED3.1 (A); no longer LED3.2 (A)
- net at R12.1: now also LED2.1 (A); no longer LED2.2 (A)
Changed lines of the file:
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@@
 	)
 	(symbol
-		(lib_id "Device:LED_Small")
+		(lib_id "Transit:Kento_LED0805_C229x")
 		(at 273.05 148.59 180)
 		(unit 1)
@@
 			)
 		)
-		(property "Sim.Pins" "1=K 2=A"
+		(property "Sim.Pins" "1=A 2=K"
 			(at 273.05 148.59 0)
 			(hide yes)
@@
 	)
 	(symbol
-		(lib_id "Device:LED_Small")
+		(lib_id "Transit:Kento_LED0805_C229x")
 		(at 278.13 33.02 90)
 		(unit 1)
@@
 			)
 		)
-		(property "Sim.Pins" "1=K 2=A"
+		(property "Sim.Pins" "1=A 2=K"
 			(at 278.13 33.02 0)
 			(hide yes)
@@
 	)
 	(symbol
-		(lib_id "Device:LED_Small")
+		(lib_id "Transit:Kento_LED0805_C229x")
 		(at 273.05 123.19 180)
 		(unit 1)
@@
 			)
 		)
-		(property "Sim.Pins" "1=K 2=A"
+		(property "Sim.Pins" "1=A 2=K"
 			(at 273.05 123.19 0)
 			(hide yes)

Commit message: Update BOM, remove VLED bulk capacitors, add Rev C to silkscreen
Parts:
- C11: LCSC Part C45783 -> C380338
- C12, C13, C16, C9: symbol EasyEDA:CL21B106KOQNNNE -> EasyEDA:FCC0805X106K100FT; LCSC Part C15849 -> C26413
- C2, C5, C6, C8: symbol EasyEDA:CL21B106KOQNNNE -> EasyEDA:FCC0805X106K100FT; LCSC Part C95841 -> C5137471
- C7: symbol EasyEDA:CL21B106KOQNNNE -> EasyEDA:FCC0805X106K100FT
- U1: value ESP32-C3-MINI-1 -> ESP32-C3-MINI-1-H4X; LCSC C2838502 -> C41349510
Changed lines of the file:
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@@
 	)
 	(symbol
-		(lib_name "CL21B106KOQNNNE_2")
-		(lib_id "EasyEDA:CL21B106KOQNNNE")
+		(lib_name "FCC0805X106K100FT_2")
+		(lib_id "EasyEDA:FCC0805X106K100FT")
 		(at 66.04 120.65 90)
 		(mirror x)
@@
 			)
 		)
-		(property "Datasheet" "https://www.lcsc.com/datasheet/C15849.pdf"
+		(property "Datasheet" "https://www.lcsc.com/product-detail/C26413.html"
 			(at 78.74 120.65 0)
 			(hide yes)
@@
 			)
 		)
-		(property "Description" "1uF ±10% 50V Ceramic Capacitor X5R 0603"
+		(property "Description" "1uF ±10% 10V Ceramic Capacitor X5R 0603"
 			(at 66.04 120.65 0)
 			(hide yes)
@@
 			)
 		)
-		(property "LCSC Part" "C15849"
+		(property "LCSC Part" "C26413"
 			(at 81.28 120.65 0)
 			(hide yes)
@@
 	)
 	(symbol
-		(lib_name "CL21B106KOQNNNE_5")
-		(lib_id "EasyEDA:CL21B106KOQNNNE")
+		(lib_name "FCC0805X106K100FT_5")
+		(lib_id "EasyEDA:FCC0805X106K100FT")
 		(at 267.97 25.4 270)
 		(unit 1)
@@
 			)
 		)
-		(property "Datasheet" "https://lcsc.com/product-detail/Multilayer-Ceramic-Capacitors-MLCC-SMD-SMT_SAMSUNG_CL21B106KOQNNNE_10uF-106-10-16V_C95841.html"
+		(property "Datasheet" "https://www.lcsc.com/product-detail/C5137471.html"
 			(at 255.27 25.4 0)
 			(hide yes)
@@
 			)
 		)
-		(property "Description" "10uF ±10% 25V Ceramic Capacitor X5R 0805"
+		(property "Description" "10uF ±10% 10V Ceramic Capacitor X5R 0805"
 			(at 267.97 25.4 0)
 			(hide yes)
@@
 			)
 		)
-		(property "LCSC Part" "C95841"
+		(property "LCSC Part" "C5137471"
 			(at 252.73 25.4 0)
 			(hide yes)
@@
 	)
 	(symbol
-		(lib_name "CL21B106KOQNNNE_4")
-		(lib_id "EasyEDA:CL21B106KOQNNNE")
+		(lib_name "FCC0805X106K100FT_4")
+		(lib_id "EasyEDA:FCC0805X106K100FT")
 		(at 219.71 63.5 90)
 		(mirror x)
@@
 			)
 		)
-		(property "Value" "ESP32-C3-MINI-1"
+		(property "Value" "ESP32-C3-MINI-1-H4X"
 			(at 64.008 39.116 0)
 			(show_name no)
@@
 			)
 		)
-		(property "LCSC" "C2838502"
+		(property "LCSC" "C41349510"
 			(at 62.23 66.04 0)
 			(hide yes)
@@
 	)
 	(symbol
-		(lib_name "CL21B106KOQNNNE_4")
-		(lib_id "EasyEDA:CL21B106KOQNNNE")
+		(lib_name "FCC0805X106K100FT_4")
+		(lib_id "EasyEDA:FCC0805X106K100FT")
 		(at 226.06 63.5 90)
 		(mirror x)
@@
 			)
 		)
-		(property "Datasheet" "https://lcsc.com/product-detail/Multilayer-Ceramic-Capacitors-MLCC-SMD-SMT_SAMSUNG_CL21B106KOQNNNE_10uF-106-10-16V_C95841.html"
+		(property "Datasheet" "https://www.lcsc.com/product-detail/C5137471.html"
 			(at 238.76 63.5 0)
 			(hide yes)
@@
 			)
 		)
-		(property "Description" "10uF ±10% 25V Ceramic Capacitor X5R 0805"
+		(property "Description" "10uF ±10% 10V Ceramic Capacitor X5R 0805"
 			(at 226.06 63.5 0)
 			(hide yes)
@@
 			)
 		)
-		(property "LCSC Part" "C95841"
+		(property "LCSC Part" "C5137471"
 			(at 241.3 63.5 0)
 			(hide yes)
@@
 	)
 	(symbol
-		(lib_name "CL21B106KOQNNNE_3")
-		(lib_id "EasyEDA:CL21B106KOQNNNE")
+		(lib_name "FCC0805X106K100FT_3")
+		(lib_id "EasyEDA:FCC0805X106K100FT")
 		(at 264.16 58.42 0)
 		(unit 1)
@@
 			)
 		)
-		(property "Datasheet" "https://www.lcsc.com/datasheet/C15849.pdf"
+		(property "Datasheet" "https://www.lcsc.com/product-detail/C26413.html"
 			(at 264.16 71.12 0)
 			(hide yes)
@@
 			)
 		)
-		(property "Description" "1uF ±10% 50V Ceramic Capacitor X5R 0603"
+		(property "Description" "1uF ±10% 10V Ceramic Capacitor X5R 0603"
 			(at 264.16 58.42 0)
 			(hide yes)
@@
 			)
 		)
-		(property "LCSC Part" "C15849"
+		(property "LCSC Part" "C26413"
 			(at 264.16 73.66 0)
 			(hide yes)
@@
 	)
 	(symbol
-		(lib_name "CL21B106KOQNNNE_4")
-		(lib_id "EasyEDA:CL21B106KOQNNNE")
+		(lib_name "FCC0805X106K100FT_4")
+		(lib_id "EasyEDA:FCC0805X106K100FT")
 		(at 227.33 25.4 90)
 		(mirror x)
@@
 			)
 		)
-		(property "Datasheet" "https://lcsc.com/product-detail/Multilayer-Ceramic-Capacitors-MLCC-SMD-SMT_SAMSUNG_CL21B106KOQNNNE_10uF-106-10-16V_C95841.html"
+		(property "Datasheet" "https://www.lcsc.com/product-detail/C5137471.html"
 			(at 240.03 25.4 0)
 			(hide yes)
@@
 			)
 		)
-		(property "Description" "10uF ±10% 25V Ceramic Capacitor X5R 0805"
+		(property "Description" "10uF ±10% 10V Ceramic Capacitor X5R 0805"
 			(at 227.33 25.4 0)
 			(hide yes)
@@
 			)
 		)
-		(property "LCSC Part" "C95841"
+		(property "LCSC Part" "C5137471"
 			(at 242.57 25.4 0)
 			(hide yes)
@@
 	)
 	(symbol
-		(lib_name "CL21B106KOQNNNE_2")
-		(lib_id "EasyEDA:CL21B106KOQNNNE")
+		(lib_name "FCC0805X106K100FT_2")
+		(lib_id "EasyEDA:FCC0805X106K100FT")
 		(at 25.4 120.65 270)
 		(unit 1)
@@
 			)
 		)
-		(property "Datasheet" "https://www.lcsc.com/datasheet/C15849.pdf"
+		(property "Datasheet" "https://www.lcsc.com/product-detail/C26413.html"
 			(at 12.7 120.65 0)
 			(hide yes)
@@
 			)
 		)
-		(property "Description" "1uF ±10% 50V Ceramic Capacitor X5R 0603"
+		(property "Description" "1uF ±10% 10V Ceramic Capacitor X5R 0603"
 			(at 25.4 120.65 0)
 			(hide yes)
@@
 			)
 		)
-		(property "LCSC Part" "C15849"
+		(property "LCSC Part" "C26413"
 			(at 10.16 120.65 0)
 			(hide yes)
@@
 	)
 	(symbol
-		(lib_id "EasyEDA:CL21B106KOQNNNE")
+		(lib_id "EasyEDA:FCC0805X106K100FT")
 		(at 234.95 109.22 270)
 		(unit 1)
@@
 			)
 		)
-		(property "Datasheet" "https://www.lcsc.com/datasheet/C15849.pdf"
+		(property "Datasheet" "https://www.lcsc.com/product-detail/C26413.html"
 			(at 222.25 109.22 0)
 			(hide yes)
@@
 			)
 		)
-		(property "Description" "1uF ±10% 50V Ceramic Capacitor X5R 0603"
+		(property "Description" "1uF ±10% 10V Ceramic Capacitor X5R 0603"
 			(at 234.95 109.22 0)
 			(hide yes)
@@
 			)
 		)
-		(property "LCSC Part" "C15849"
+		(property "LCSC Part" "C26413"
 			(at 219.71 109.22 0)
 			(hide yes)
@@
 			)
 		)
-		(property "Datasheet" "https://www.lcsc.com/datasheet/C45783.pdf"
+		(property "Datasheet" "https://www.lcsc.com/product-detail/C380338.html"
 			(at 158.75 116.84 0)
 			(hide yes)
@@
 			)
 		)
-		(property "Description" "22uF ±20% 25V Ceramic Capacitor X5R 0805"
+		(property "Description" "22uF ±20% 10V Ceramic Capacitor X5R 0805"
 			(at 146.05 116.84 0)
 			(hide yes)
@@
 			)
 		)
-		(property "LCSC Part" "C45783"
+		(property "LCSC Part" "C380338"
 			(at 161.29 116.84 0)
 			(hide yes)
@@
 	)
 	(symbol
-		(lib_name "CL21B106KOQNNNE_1")
-		(lib_id "EasyEDA:CL21B106KOQNNNE")
+		(lib_name "FCC0805X106K100FT_1")
+		(lib_id "EasyEDA:FCC0805X106K100FT")
 		(at 49.53 25.4 0)
 		(unit 1)
@@
 			)
 		)
-		(property "Datasheet" "https://lcsc.com/product-detail/Multilayer-Ceramic-Capacitors-MLCC-SMD-SMT_SAMSUNG_CL21B106KOQNNNE_10uF-106-10-16V_C95841.html"
+		(property "Datasheet" "https://www.lcsc.com/product-detail/C5137471.html"
 			(at 49.53 38.1 0)
 			(hide yes)
@@
 			)
 		)
-		(property "Description" "10uF ±10% 25V Ceramic Capacitor X5R 0805"
+		(property "Description" "10uF ±10% 10V Ceramic Capacitor X5R 0805"
 			(at 49.53 25.4 0)
 			(hide yes)
@@
 			)
 		)
-		(property "LCSC Part" "C95841"
+		(property "LCSC Part" "C5137471"
 			(at 49.53 40.64 0)
 			(hide yes)

Commit message: Update silkscreen, remove tp8, fix stale tp values
Parts:
- removed TP8: +VBUS, TestPoint:TestPoint_Keystone_5000-5004_Miniature, symbol Connector:TestPoint
- TP5: value Ambient-Light-SNS -> VBUS_RAW
- TP6: value Ambient-Light-SNS -> FERRY
- TP7: value Ambient-Light-SNS -> RAIL
Changed lines of the file:
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@@
 	)
 	(junction
-		(at 186.69 74.93)
-		(diameter 0)
-		(color 0 0 0 0)
-	)
-	(junction
 		(at 195.58 27.94)
 		(diameter 0)
@@
 	(wire
 		(pts
-			(xy 186.69 77.47) (xy 186.69 74.93)
+			(xy 186.69 71.12) (xy 186.69 77.47)
 		)
 		(stroke
@@
 	(wire
 		(pts
-			(xy 186.69 74.93) (xy 186.69 71.12)
-		)
-		(stroke
-			(width 0)
-			(type default)
-		)
-	)
-	(wire
-		(pts
 			(xy 60.96 27.94) (xy 62.23 27.94)
 		)
@@
 			)
 		)
-		(property "Value" "Ambient-Light-SNS"
+		(property "Value" "FERRY"
 			(at 71.628 151.638 0)
 			(hide yes)
@@
 	)
 	(symbol
-		(lib_id "Connector:TestPoint")
-		(at 186.69 74.93 270)
-		(unit 1)
-		(body_style 1)
-		(exclude_from_sim no)
-		(in_bom yes)
-		(on_board yes)
-		(in_pos_files yes)
-		(dnp yes)
-		(property "Reference" "TP8"
-			(at 193.04 74.93 90)
-			(show_name no)
-			(do_not_autoplace no)
-			(effects
-				(font
-					(size 1.27 1.27)
-				)
-				(justify left)
-			)
-		)
-		(property "Value" "+VBUS"
-			(at 192.278 73.152 0)
-			(hide yes)
-			(show_name no)
-			(do_not_autoplace no)
-			(effects
-				(font
-					(size 1.27 1.27)
-				)
-				(justify left)
-			)
-		)
-		(property "Footprint" "TestPoint:TestPoint_Keystone_5000-5004_Miniature"
-			(at 186.69 80.01 0)
-			(hide yes)
-			(show_name no)
-			(do_not_autoplace no)
-			(effects
-				(font
-					(size 1.27 1.27)
-				)
-			)
-		)
-		(property "Datasheet" ""
-			(at 186.69 80.01 0)
-			(hide yes)
-			(show_name no)
-			(do_not_autoplace no)
-			(effects
-				(font
-					(size 1.27 1.27)
-				)
-			)
-		)
-		(property "Description" "TP +VBUS"
-			(at 186.69 74.93 0)
-			(hide yes)
-			(show_name no)
-			(do_not_autoplace no)
-			(effects
-				(font
-					(size 1.27 1.27)
-				)
-			)
-		)
-		(pin "1"
-		)
-		(instances
-			(project "transit"
-				(path "/3763eade-a8c8-4ec0-9cf2-9db4442b4ee5"
-					(reference "TP8")
-					(unit 1)
-				)
-			)
-		)
-	)
-	(symbol
 		(lib_name "FCC0805X106K100FT_2")
 		(lib_id "EasyEDA:FCC0805X106K100FT")
@@
 			)
 		)
-		(property "Value" "Ambient-Light-SNS"
+		(property "Value" "RAIL"
 			(at 72.898 160.528 0)
 			(hide yes)
@@
 			)
 		)
-		(property "Value" "Ambient-Light-SNS"
+		(property "Value" "VBUS_RAW"
 			(at 176.022 32.258 0)
 			(hide yes)

Commit message: Update README, fix typos
Other:
- title: Seattle Transit -> Seattle Transit Live
Changed lines of the file:
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@@
 	(paper "A4")
 	(title_block
-		(title "Seattle Transit")
-		(date "2026-05-06")
-		(rev "B")
+		(title "Seattle Transit Live")
+		(date "2026-07-25")
+		(rev "C")
 		(company "Salt River Labs")
 	)
@@
 	)
 	(junction
-		(at 148.59 104.14)
-		(diameter 0)
-		(color 0 0 0 0)
-	)
-	(junction
 		(at 262.89 60.96)
 		(diameter 0)
@@
 	(wire
 		(pts
-			(xy 148.59 104.14) (xy 148.59 101.6)
+			(xy 148.59 101.6) (xy 148.59 106.68)
 		)
 		(stroke
@@
 	(wire
 		(pts
-			(xy 147.32 104.14) (xy 148.59 104.14)
-		)
-		(stroke
-			(width 0)
-			(type default)
-		)
-	)
-	(wire
-		(pts
 			(xy 276.86 123.19) (xy 275.59 123.19)
 		)
@@
 		)
 		(stroke
-			(width 0)
-			(type default)
-		)
-	)
-	(wire
-		(pts
-			(xy 148.59 104.14) (xy 148.59 106.68)
-		)
-		(stroke
